File: PCB/V1.0/CREPP.io.kicad_pcb (KiCad board)
At the start: 2 copper layers, 101.9 x 139.4 mm, 100 parts, among them J1 Screw_Terminal_01x04, J10 Right_Connector, J11 Right_Connector, J12 Right_Connector, J13 Conn_02x04_Odd_Even, J14 OLED_SOCKET, J15 Conn_02x04_Odd_Even, J16 I2C_Selector, J17 Conn_02x04_Odd_Even, J18 Conn_02x04_Odd_Even, J19 Analog_Inputs, J2 HC-SR04_VIRTUAL, J20 GND_Analog, J21 +3.3V_Analog, J22 OLED_SOCKET_VIRTUAL, J23 HC-SR, J24 BME_VIRTUAL, J25 BME, J26 Addr_Selector, J27 SIG_HCSR04, J28 SIG_HC-05, J29 Conn_01x06_Socket, J3 Conn_02x04_Odd_Even, J30 Servo, J31 HC-05_VIRTUAL, J32 Power_Servo_Selector, J33 Screw_Terminal_01x02, J34 Sig_Servo, J35 SPI_Connector, J36 Power_Selector, J37 Sig_MOSFET, J4 Right_Connector, J5 Right_Connector, J6 Right_Connector, J7 Left_Connector, J8 Right_Connector, J9 Right_Connector, Q1 IRF520, SW1 SW_Left, SW2 SW_Up, SW3 SW_Right, SW4 SW_Down, T1 TestPoint, T4 TestPoint, U1 ADS1115IDGS, U14 DS1307+, U2 PC817, U3 ESP-12E_VIRTUAL, Y2 16MHz

Commit message: Test URl MD
Parts:
- removed J2: HC-SR04_VIRTUAL, Connector_PinSocket_2.54mm:PinSocket_1x04_P2.54mm_Vertical
- removed J22: OLED_SOCKET_VIRTUAL, Connector_PinSocket_2.54mm:PinSocket_1x04_P2.54mm_Vertical
- removed J31: HC-05_VIRTUAL, Connector_PinSocket_2.54mm:PinSocket_1x04_P2.54mm_Vertical
- removed JP1 (x20): J2.54MM, Connector_PinHeader_2.54mm:PinHeader_2x01_P2.54mm_Vertical
- removed U3: ESP-12E_VIRTUAL, RF_Module:ESP-12E
- R11: value LDR07 -> ${REFERENCE}
- moved J21 44.4 mm to (100.9, 160.2)
- moved Q1 44.4 mm to (122.0, 84.9)
- moved R4 44.4 mm to (76.5, 131.5)
- moved RV1 44.4 mm to (58.0, 79.4)
- moved C17 44.4 mm to (70.0, 82.2)
- moved D5 44.4 mm to (127.1, 90.3)
- moved H2 44.4 mm to (51.6, 39.3)
- moved H3 44.4 mm to (49.3, 166.3)
- moved J10 44.4 mm to (116.1, 124.1)
- moved J26 44.4 mm to (49.3, 150.5)
- moved J32 44.4 mm to (126.3, 69.2)
- moved J7 44.4 mm to (57.5, 144.2)
- moved J8 44.4 mm to (126.3, 124.1)
- moved R12 44.4 mm to (113.8, 96.6)
- moved R14 44.4 mm to (124.0, 90.1)
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Other:
- board text removed: "PCB3D_BR_BOARD"
- board text removed: "PCB3D_TL_BOARD"
