File: PCB/V1.1/CREPP.io.kicad_pcb (KiCad board)
At the start: 2 copper layers, 101.9 x 139.4 mm, 79 parts, among them J1 Screw_Terminal_01x04, J10 Right_Connector, J11 Right_Connector, J12 Right_Connector, J13 Conn_02x04_Odd_Even, J14 OLED_SOCKET, J15 Conn_02x04_Odd_Even, J16 I2C_Selector, J17 Conn_02x04_Odd_Even, J18 Conn_02x04_Odd_Even, J19 Analog_Inputs, J20 GND_Analog, J21 +3.3V_Analog, J23 HC-SR, J25 BME, J26 Addr_Selector, J27 SIG_HCSR04, J28 SIG_HC-05, J29 Conn_01x06_Socket, J3 Conn_02x04_Odd_Even, J30 Servo, J32 Power_Servo_Selector, J33 Screw_Terminal_01x02, J34 Sig_Servo, J35 SPI_Connector, J36 Power_Selector, J37 Sig_MOSFET, J4 Right_Connector, J5 Right_Connector, J6 Right_Connector, J7 Left_Connector, J8 Right_Connector, J9 Right_Connector, Q1 IRF520, Q2 2N7000, SW1 SW_Left, SW2 SW_Up, SW3 SW_Right, SW4 SW_Down, SW5 SW_Left, T1 TestPoint, T4 TestPoint, U1 ADS1115IDGS, U14 DS1307+, U2 PC817, Y2 16MHz

Commit message: Test URl MD
Parts:
- moved J12 30.7 mm to (160.6, 108.0)
- moved R27 30.7 mm to (141.0, 73.5)
- moved SW3 30.7 mm to (154.8, 49.0)
- moved U2 30.7 mm to (173.4, 78.7)
- moved J1 30.7 mm to (189.2, 80.1)
- moved J13 30.7 mm to (168.2, 92.2)
- moved J15 30.7 mm to (168.2, 97.3)
- moved J17 30.7 mm to (187.7, 121.7)
- moved J30 30.7 mm to (176.8, 52.8)
- moved R5 30.7 mm to (190.9, 148.5)
- moved R9 30.7 mm to (171.2, 70.4)
- moved C1 30.7 mm to (148.9, 136.6)
- moved J35 30.7 mm to (105.7, 105.4)
- moved R4 30.7 mm to (131.1, 115.3)
- moved U1 30.7 mm to (151.9, 135.3)
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Other:
- board text removed: "PCB3D_BR_BOARD"
- board text removed: "PCB3D_TL_BOARD"

Commit message: Update
Other:
- board text added: "Remove D8 Jumper or press Left button when uploading program"
- board text removed: "Remove D8 Jumper or press Left button when sending program"
Changed lines of the file:
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@@
 		(allow_soldermask_bridges_in_footprints no)
 		(pcbplotparams
-			(layerselection 0x0000020_7ffffffe)
-			(plot_on_all_layers_selection 0x0009020_00000000)
+			(layerselection 0x00010fc_ffffffff)
+			(plot_on_all_layers_selection 0x0001000_00000000)
 			(disableapertmacros no)
 			(usegerberextensions no)
@@
 			(sketchpadsonfab yes)
 			(subtractmaskfromsilk no)
-			(outputformat 4)
+			(outputformat 1)
 			(mirror no)
 			(drillshape 0)
@@
 		)
 		(property "Value" "270"
-			(at 8.128 12.362 0)
+			(at 5.395406 0.557811 0)
 			(layer "F.Fab")
 			(effects
@@
 		)
 		(fp_text user "${REFERENCE}"
-			(at 3.81 0 0)
+			(at 1.788606 -0.407389 0)
 			(layer "F.Fab")
 			(effects
@@
 		)
 		(fp_text user "${REFERENCE}"
-			(at 1.45 4.999999 0)
+			(at 3.109406 5.028211 0)
 			(layer "F.Fab")
 			(effects
@@
 		)
 		(property "Value" "Servo"
-			(at 0 7.41 0)
+			(at 0.061406 -2.251189 0)
 			(layer "F.Fab")
 			(effects
@@
 		)
 		(property "Value" "LED"
-			(at 1.27 3.96 180)
+			(at 0.802194 1.321789 180)
 			(layer "F.Fab")
 			(effects
@@
 			(at -1.27 38.33 180)
 			(layer "F.Fab")
+			(hide yes)
 			(effects
 				(font
@@
 		)
 		(property "Value" "270"
-			(at 3.81 2.37 180)
+			(at -2.804606 -0.024411 180)
 			(layer "F.Fab")
 			(effects
@@
 		)
 		(property "Value" "I2C_Selector"
-			(at 1.27 7.41 -90)
+			(at 5.131789 2.906206 0)
 			(layer "F.Fab")
 			(effects
@@
 		)
 		(property "Value" "Screw_Terminal_01x02"
-			(at 2.5 5.66 -90)
+			(at 9.115789 2.398206 0)
 			(layer "F.Fab")
 			(effects
@@
 		)
 		(property "Value" "10k"
-			(at 3.81 2.37 0)
+			(at 5.598606 0.608611 0)
 			(layer "F.Fab")
 			(effects
@@
 		)
 		(fp_text user "${REFERENCE}"
-			(at 3.81 0 0)
+			(at 1.737806 -0.356589 0)
 			(layer "F.Fab")
 			(effects
@@
 			(at -4.424 3.212 -90)
 			(layer "F.Fab")
+			(hide yes)
 			(effects
 				(font
@@
 		)
 		(property "Value" "1k"
-			(at 3.81 2.37 -90)
+			(at 5.588989 0.417006 -90)
 			(layer "F.Fab")
 			(effects
@@
 		)
 		(fp_text user "${REFERENCE}"
-			(at 3.81 0 -90)
+			(at 2.286989 -0.344994 -90)
 			(layer "F.Fab")
 			(effects
@@
 			(at 0 1.55 0)
 			(layer "F.Fab")
+			(hide yes)
 			(effects
 				(font
@@
 		)
 		(property "Value" "LED"
-			(at 1.27 3.96 180)
+			(at 0.751394 1.372589 180)
 			(layer "F.Fab")
 			(effects
@@
 		)
 		(property "Value" "PC817"
-			(at 3.81 4.87 0)
+			(at 3.851006 2.977411 0)
 			(layer "F.Fab")
 			(effects
@@
 			(at 0 9.95 0)
 			(layer "F.Fab")
+			(hide yes)
 			(effects
 				(font
@@
 			(at -1.27 38.33 180)
 			(layer "F.Fab")
+			(hide yes)
 			(effects
 				(font
@@
 		)
 		(property "Value" "LED"
-			(at 1.27 3.96 -90)
+			(at -0.811811 0.213806 0)
 			(layer "F.Fab")
 			(effects
@@
 		)
 		(fp_text user "K"
-			(at -2.032 1.016 0)
+			(at 1.728189 2.042606 0)
 			(layer "F.Fab")
 			(effects
@@
 		)
 		(property "Value" "10k"
-			(at 3.81 2.37 0)
+			(at 5.598606 0.608611 0)
 			(layer "F.Fab")
 			(effects
@@
 		)
 		(fp_text user "${REFERENCE}"
-			(at 3.81 0 0)
+			(at 1.687006 -0.407389 0)
 			(layer "F.Fab")
 			(effects
@@
 		)
 		(property "Value" "Conn_01x06_Socket"
-			(at 0 15.47 90)
+			(at -2.845789 7.101394 180)
 			(layer "F.Fab")
 			(effects
@@
 			(at 0 7.41 0)
 			(layer "F.Fab")
+			(hide yes)
 			(effects
 				(font
@@
 		)
 		(property "Value" "10k"
-			(at 3.81 2.37 0)
+			(at 5.598606 0.659411 0)
 			(layer "F.Fab")
 			(effects
@@
 		)
 		(fp_text user "${REFERENCE}"
-			(at 3.81 0 0)
+			(at 1.737806 -0.305789 0)
 			(layer "F.Fab")
 			(effects
@@
 		)
 		(property "Value" "270"
-			(at 3.81 2.37 180)
+			(at 2.148394 -0.583211 180)
 			(layer "F.Fab")
 			(effects
@@
 		)
 		(fp_text user "${REFERENCE}"
-			(at 3.81 0 180)
+			(at 5.856794 0.381989 180)
 			(layer "F.Fab")
 			(effects
@@
 			(at 0 7.41 0)
 			(layer "F.Fab")
+			(hide yes)
 			(effects
 				(font
@@
 		)
 		(property "Value" "10k"
-			(at 3.81 2.37 0)
+			(at 5.598606 0.659411 0)
 			(layer "F.Fab")
 			(effects
@@
 		)
 		(fp_text user "${REFERENCE}"
-			(at 3.81 0 0)
+			(at 2.195006 -0.356589 0)
 			(layer "F.Fab")
 			(effects
@@
 		)
 		(property "Value" "10k"
-			(at 3.81 2.37 180)
+			(at 2.072194 -0.557811 180)
 			(layer "F.Fab")
 			(effects
@@
 		)
 		(fp_text user "${REFERENCE}"
-			(at 3.81 0 180)
+			(at 5.475794 0.458189 180)
 			(layer "F.Fab")
 			(effects
@@
 		)
 		(property "Value" "270"
-			(at 3.81 2.37 90)
+			(at 2.285011 -0.417006 90)
 			(layer "F.Fab")
 			(effects
@@
 		)
 		(fp_text user "${REFERENCE}"
-			(at 3.81 0 90)
+			(at 5.282211 0.344994 90)
 			(layer "F.Fab")
 			(effects
@@
 		)
 		(property "Value" "Screw_Terminal_01x04"
-			(at 7.62 5.66 -90)
+			(at 8.054589 5.821006 -90)
 			(layer "F.Fab")
 			(effects
@@
 		)
 		(property "Value" "270"
-			(at 3.81 2.37 0)
+			(at 5.395406 0.557811 0)
 			(layer "F.Fab")
 			(effects
@@
 		)
 		(fp_text user "${REFERENCE}"
-			(at 3.81 0 0)
+			(at 1.788606 -0.407389 0)
 			(layer "F.Fab")
 			(effects
@@
 		)
 		(property "Value" "270"
-			(at 3.81 2.37 0)
+			(at 5.293806 0.608611 0)
 			(layer "F.Fab")
 			(effects
@@
 		)
 		(fp_text user "${REFERENCE}"
-			(at 3.81 0 0)
+			(at 1.737806 -0.407389 0)
 			(layer "F.Fab")
 			(effects
@@
 			(at 0 4.87 -90)
 			(layer "F.Fab")
+			(hide yes)
 			(effects
 				(font
@@
 		)
 		(property "Value" "10k"
-			(at 3.81 2.37 0)
+			(at 5.344606 0.507011 0)
 			(layer "F.Fab")
 			(effects
@@
 		)
 		(fp_text user "${REFERENCE}"
-			(at 3.81 0 0)
+			(at 2.347406 -0.305789 0)
 			(layer "F.Fab")
 			(effects
@@
 		)
 		(property "Value" "IRF520"
-			(at 2.54 2.5 -90)
+			(at 2.54 2.266606 -90)
 			(layer "F.Fab")
 			(effects
@@
 		)
 		(fp_text user "${REFERENCE}"
-			(at 2.54 -4.27 -90)
+			(at 6.782989 -0.628994 0)
 			(layer "F.Fab")
 			(effects
@@
 		)
 		(property "Value" "OLED_SOCKET"
-			(at 0 10.39 90)
+			(at -2.591789 4.256594 180)
 			(layer "F.Fab")
 			(effects
@@
 			(at 0 4.87 90)
 			(layer "F.Fab")
+			(hide yes)
 			(effects
 				(font
@@
 		)
 		(property "Value" "Sig_Servo"
-			(at 0 2.33 0)
+			(at -1.310194 2.132611 0)
 			(layer "F.Fab")
 			(effects
@@
 		)
 		(property "Value" "10k"
-			(at 3.81 2.37 0)
+			(at 5.598606 0.608611 0)
 			(layer "F.Fab")
 			(effects
@@
 		)
 		(fp_text user "${REFERENCE}"
-			(at 3.81 0 0)
+			(at 1.737806 -0.407389 0)
 			(layer "F.Fab")
 			(effects
@@
 		)
 		(property "Value" "LED"
-			(at 1.27 3.96 180)
+			(at 0.852994 1.270989 180)
 			(layer "F.Fab")
 			(effects
@@
 		)
 		(property "Value" "10k"
-			(at 3.81 2.37 -90)
+			(at 5.284189 0.315406 -90)
 			(layer "F.Fab")
 			(effects
@@
 		)
 		(fp_text user "${REFERENCE}"
-			(at 3.81 0 -90)
+			(at 1.829789 -0.243394 -90)
 			(layer "F.Fab")
 			(effects
@@
 		)
 		(property "Value" "1k"
-			(at 3.81 2.37 180)
+			(at 1.970594 -0.405411 180)
 			(layer "F.Fab")
 			(effects
@@
 		)
 		(fp_text user "${REFERENCE}"
-			(at 3.81 0 180)
+			(at 5.221794 0.356589 180)
 			(layer "F.Fab")
 			(effects
@@
 		)
 		(property "Value" "10k"
-			(at 3.81 2.37 0)
+			(at 5.547806 0.608611 0)
 			(layer "F.Fab")
 			(effects
@@
 		)
 		(fp_text user "${REFERENCE}"
-			(at 3.81 0 0)
+			(at 2.144206 -0.305789 0)
 			(layer "F.Fab")
 			(effects
@@
 			(at 0 1.55 0)
 			(layer "F.Fab")
+			(hide yes)
 			(effects
 				(font
@@
 		)
 		(property "Value" "2N7000"
-			(at 1.27 2.79 180)
+			(at 1.157794 2.434989 180)
 			(layer "F.Fab")
 			(effects
@@
 		)
 	)
-	(gr_text "Remove D8 Jumper or press Left button when sending program"
+	(gr_text "Remove D8 Jumper or press Left button when uploading program"
 		(at 116.930994 153.264589 0)
 		(layer "F.SilkS")
