File: PCB/CCR/CCR.kicad_sch (KiCad schematic)
At the start: 5 parts, among them U1 ATmega328P-A

Commit message: Update of BME and OLED
Parts:
- added D1, D2: LED, LED_SMD:LED_0603_1608Metric, symbol Device:LED
- added H5, H6: MountingHole, MountingHole:MountingHole_3.2mm_M3, symbol Mechanical:MountingHole
- added J1: Connecteur_SMA, CREPP_SMA:SMA_Amphenol_132289_EdgeMount, symbol CREPP_Connectors_SMA:Connecteur_SMA
- added J2: USB_C_Receptacle, CREPP_Connectors_USB:USB_C_Receptacle_GCT_USB4085, symbol CREPP_Connectors_USB_C:USB_C_Receptacle
- added OLED1: ~, CREPP_Screens:SSD1306_OLED_Display_VIRTUAL_128_64, symbol CREPP_Screens:OLED_SSD1306_0.96
- added R1, R2: 270, Resistor_SMD:R_0603_1608Metric, symbol Device:R
- added SW1: RotaryEncoder_Switch, CREPP_RotaryEncoders:RotaryEncoder, symbol CREPP_RotaryEncoders:RotaryEncoder_Switch
- added U2: NRF24L01, Package_DFN_QFN:QFN-20-1EP_4x4mm_P0.5mm_EP2.5x2.5mm, symbol RF:NRF24L01
- added U3: MPU-6050, Sensor_Motion:InvenSense_QFN-24_4x4mm_P0.5mm, symbol CREPP_Accelerometers:MPU-6050
- added U4: COM-09032, CREPP_Joysticks_SW:XDCR_COM-09032, symbol CREPP_Joysticks:COM-09032_JOYSTICK
- added U5: TP4056, CREPP_BMS:SOP127P600X175-9N, symbol CREPP_BMS:TP4056
Connections:
- new net: D1.1 (K), U5.6 (~{STDBY})
- new net: D1.2 (A), R1.2
- new net: D2.1 (K), U5.7 (~{CHRG})
- new net: D2.2 (A), R2.2
- new net: J2.A1 (GND), J2.A12 (GND), J2.B1 (GND), J2.B12 (GND)
- new net: J2.A4 (VBUS), J2.A9 (VBUS), J2.B4 (VBUS), J2.B9 (VBUS)
- new net: U4.S1 (SHIELD), U4.S2 (SHIELD), U4.S3 (SHIELD), U4.S4 (SHIELD)
Other:
- removed sheet UserActions
