File: PCB/CCR/Modules/IMU.kicad_sch (KiCad schematic)
At the start: 1 part, among them U4 MPU-6050

Commit message: Update of BME and OLED
Parts:
- removed U4: MPU-6050, Sensor_Motion:InvenSense_QFN-24_4x4mm_P0.5mm, symbol Sensor_Motion:MPU-6050
Changed lines of the file:
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@@
-		)
-	)
-	(symbol
-		(lib_id "Sensor_Motion:MPU-6050")
-		(at 43.18 71.12 0)
-		(unit 1)
-		(exclude_from_sim no)
-		(in_bom yes)
-		(on_board yes)
-		(dnp no)
-		(fields_autoplaced yes)
-		(property "Reference" "U4"
-			(at 45.3741 87.63 0)
-			(effects
-				(font
-					(size 1.27 1.27)
-				)
-				(justify left)
-			)
-		)
-		(property "Value" "MPU-6050"
-			(at 45.3741 90.17 0)
-			(effects
-				(font
-					(size 1.27 1.27)
-				)
-				(justify left)
-			)
-		)
-		(property "Footprint" "Sensor_Motion:InvenSense_QFN-24_4x4mm_P0.5mm"
-			(at 43.18 91.44 0)
-			(effects
-				(font
-					(size 1.27 1.27)
-				)
-				(hide yes)
-			)
-		)
-		(property "Datasheet" "https://invensense.tdk.com/wp-content/uploads/2015/02/MPU-6000-Datasheet1.pdf"
-			(at 43.18 74.93 0)
-			(effects
-				(font
-					(size 1.27 1.27)
-				)
-				(hide yes)
-			)
-		)
-		(property "Description" "InvenSense 6-Axis Motion Sensor, Gyroscope, Accelerometer, I2C"
-			(at 43.18 71.12 0)
-			(effects
-				(font
-					(size 1.27 1.27)
-				)
-				(hide yes)
-			)
-		)
-		(pin "23"
-		)
-		(pin "10"
-		)
-		(pin "17"
-		)
-		(pin "16"
-		)
-		(pin "22"
-		)
-		(pin "1"
-		)
-		(pin "3"
-		)
-		(pin "8"
-		)
-		(pin "11"
-		)
-		(pin "13"
-		)
-		(pin "2"
-		)
-		(pin "6"
-		)
-		(pin "21"
-		)
-		(pin "24"
-		)
-		(pin "4"
-		)
-		(pin "15"
-		)
-		(pin "12"
-		)
-		(pin "19"
-		)
-		(pin "7"
-		)
-		(pin "5"
-		)
-		(pin "14"
-		)
-		(pin "18"
-		)
-		(pin "20"
-		)
-		(pin "9"
-		)
-		(instances
-			(project "CCR"
-				(path "/8bcd0d00-b75f-4070-8d50-196a2022a31c/82793622-14ac-4029-92dc-96c42c2d5609"
-					(reference "U4")
-					(unit 1)
-				)
-			)
 		)
 	)
