File: PCB/CCR/Modules/LED.kicad_sch (KiCad schematic)
At the start: 4 parts

Commit message: Update of BME and OLED
Parts:
- removed D1, D3: LED, LED_THT:LED_D5.0mm, symbol Device:LED
- removed R6, R8: 270, Resistor_THT:R_Axial_DIN0207_L6.3mm_D2.5mm_P10.16mm_Horizontal, symbol Device:R
