File: PCB/CCR/Modules/Power.kicad_sch (KiCad schematic)
At the start: 8 parts, among them J26 Servo, J29 Sig_Servo, J30 Servo, J32 Power_Servo_Selector, J33 Screw_Terminal_01x02, J34 Sig_Servo, M3 Motor_DC

Commit message: Update of BME and OLED
Parts:
- removed J26, J30: Servo, Connector_PinHeader_2.54mm:PinHeader_1x03_P2.54mm_Vertical, symbol Connector:Conn_01x03_Pin
- removed J29, J34: Sig_Servo, Connector_PinHeader_2.54mm:PinHeader_1x01_P2.54mm_Vertical, symbol Connector:Conn_01x01_Pin
- removed J32: Power_Servo_Selector, Connector_PinHeader_2.54mm:PinHeader_1x03_P2.54mm_Vertical, symbol Connector:Conn_01x03_Pin
- removed J33: Screw_Terminal_01x02, TerminalBlock_Phoenix:TerminalBlock_Phoenix_MKDS-3-2-5.08_1x02_P5.08mm_Horizontal, symbol Connector:Screw_Terminal_01x02
- removed JP30: Jumper_2.54mm_red, CREPP_Jumpers:Jumper_2.54mm_red, symbol CREPP_Jumpers:Jumper_2.54mm_red
- removed M3: Motor_DC, Connector_PinHeader_2.54mm:PinHeader_1x01_P2.54mm_Vertical, symbol Motor:Motor_DC
