File: PCB/CCR/Modules/UserActions.kicad_sch (KiCad schematic)
At the start: 10 parts, among them SW1 SW_Left, SW2 SW_Up, SW3 SW_Right, SW4 SW_Down, U10 COM-09032

Commit message: Update of BME and OLED
Parts:
- removed R1, R11, R2, R3, R4: 10k, Resistor_THT:R_Axial_DIN0207_L6.3mm_D2.5mm_P10.16mm_Horizontal, symbol Device:R
- removed SW1: SW_Left, Button_Switch_THT:SW_PUSH_6mm, symbol Switch:SW_Push
- removed SW2: SW_Up, Button_Switch_THT:SW_PUSH_6mm, symbol Switch:SW_Push
- removed SW3: SW_Right, Button_Switch_THT:SW_PUSH_6mm, symbol Switch:SW_Push
- removed SW4: SW_Down, Button_Switch_THT:SW_PUSH_6mm, symbol Switch:SW_Push
- removed U10: COM-09032, CREPP_Joysticks:XDCR_COM-09032, symbol CREPP_Joysticks:COM-09032
