File: PCB/V2.0/CREPP.io.kicad_pcb (KiCad board)
At the start: 2 copper layers, 101.9 x 139.4 mm, 82 parts, among them J1 Screw_Terminal_01x04, J10 Right_Connector, J11 Right_Connector, J12 Right_Connector, J13 Conn_02x04_Odd_Even, J14 OLED_SOCKET, J15 Conn_02x04_Odd_Even, J16 I2C_Selector, J17 Conn_02x04_Odd_Even, J18 Conn_02x04_Odd_Even, J19 Analog_Inputs, J2 HC-SR04_VIRTUAL, J20 GND_Analog, J21 +3.3V_Analog, J22 OLED_SOCKET_VIRTUAL, J23 HC-SR, J24 BME_VIRTUAL, J25 BME, J26 Addr_Selector, J27 SIG_HCSR04, J28 Conn_02x20, J3 Conn_02x04_Odd_Even, J30 Servo, J32 Power_Servo_Selector, J33 Screw_Terminal_01x02, J34 Sig_Servo, J36 Power_Selector, J37 Sig_MOSFET, J4 Conn_01x20, J5 Right_Connector, J8 Right_Connector, J9 Right_Connector, Q1 IRF520, Q2 2N7002, SW1 SW_Left, SW2 SW_Up, SW3 SW_Right, SW4 SW_Down, SW5 SW_Left, SW6 RotaryEncoder_Switch, SW7 SW_Center, T1 TestPoint, U1 ADS1115IDGS, U14 DS1307+, U2 PC817, Y2 16MHz

Commit message: Update 2.0 - IMU and NRF24 support
Parts:
- added J40: Conn_01x08_Socket, Connector_PinSocket_2.54mm:PinSocket_1x08_P2.54mm_Vertical, F.Cu at (2.03, 110.2)
- added J6: Conn_02x20, Connector_PinHeader_2.54mm:PinHeader_2x20_P2.54mm_Vertical, F.Cu at (12.4, 133.9)
- added J7: VIRTUAL_MPU6050, Connector_PinSocket_2.54mm:PinSocket_1x08_P2.54mm_Vertical, F.Cu at (2.03, 110.2)
- added U3: NRF24L01_Breakout, RF_Module:nRF24L01_Breakout, F.Cu at (215.3, 66.2)
- added U4: RP2040, Package_DFN_QFN:QFN-56-1EP_7x7mm_P0.4mm_EP3.2x3.2mm, F.Cu at (29.6, 108.7)
- J4: footprint Connector_PinSocket_2.54mm:PinSocket_2x10_P2.54mm_Vertical -> Connector_PinSocket_2.54mm:PinSocket_1x20_P2.54mm_Vertical
- J5: value Right_Connector -> Conn_01x20; footprint Connector_PinSocket_2.54mm:PinSocket_2x15_P2.54mm_Vertical -> Connector_PinSocket_2.54mm:PinSocket_1x20_P2.54mm_Vertical
- moved J24 239.4 mm to (1.78, 99.6), turned to 180 degrees
- moved J22 209.6 mm to (25.9, 55.9), turned to 90 degrees
- moved RV1 174.6 mm to (-56.4, 107.3)
- moved J14 159.1 mm to (33.4, 55.8)
- moved SW7 145.8 mm to (70.5, 95.5)
- moved J25 124.8 mm to (1.78, 99.6), turned to 180 degrees
- moved J5 122.1 mm to (20.3, 134.1)
- moved SW6 109.0 mm to (-42.9, 109.7)
- moved R1 107.4 mm to (26.2, 95.8)
- moved R2 107.4 mm to (26.2, 85.9)
- moved R3 107.4 mm to (26.2, 89.2)
- moved R4 107.4 mm to (26.2, 92.5)
- moved LDR1 99.9 mm to (11.2, 146.9)
- moved R15 92.4 mm to (33.0, 127.0)
- moved J4 89.0 mm to (38.3, 86.2), turned to 0 degrees
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Connections:
- J5 pad 1: /MCU/Pin_2 -> unconnected-(J5-Pin_1-Pad1)
- J5 pad 10: /MCU/Pin_10 -> unconnected-(J5-Pin_10-Pad10)
- J5 pad 11: /MCU/Pin_12 -> unconnected-(J5-Pin_11-Pad11)
- J5 pad 12: /MCU/Pin_12 -> unconnected-(J5-Pin_12-Pad12)
- J5 pad 13: /MCU/Pin_14 -> Net-(J5-Pin_13)
- J5 pad 14: /MCU/Pin_14 -> unconnected-(J5-Pin_14-Pad14)
- J5 pad 15: /MCU/Pin_16 -> unconnected-(J5-Pin_15-Pad15)
- J5 pad 16: /MCU/Pin_16 -> unconnected-(J5-Pin_16-Pad16)
- J5 pad 17: GND -> unconnected-(J5-Pin_17-Pad17)
- J5 pad 18: GND -> Net-(J5-Pin_18)
- J5 pad 19: /MCU/Pin_20 -> unconnected-(J5-Pin_19-Pad19)
- J5 pad 2: /MCU/Pin_2 -> unconnected-(J5-Pin_2-Pad2)
- J5 pad 20: /MCU/Pin_20 -> unconnected-(J5-Pin_20-Pad20)
- J5 pad 3: GND -> Net-(J5-Pin_3)
- J5 pad 4: GND -> unconnected-(J5-Pin_4-Pad4)
- J5 pad 5: /MCU/Pin_6 -> unconnected-(J5-Pin_5-Pad5)
- J5 pad 6: /MCU/Pin_6 -> unconnected-(J5-Pin_6-Pad6)
- J5 pad 7: /MCU/Pin_8 -> unconnected-(J5-Pin_7-Pad7)
- J5 pad 8: /MCU/Pin_8 -> Net-(J5-Pin_8)
- J5 pad 9: /MCU/Pin_10 -> unconnected-(J5-Pin_9-Pad9)
Routing:
- net +3.3V: track 491.7 -> 0.00 mm, vias 3 -> 0
- net +5V: track 406.8 -> 0.00 mm, vias 1 -> 0
- net /IO_Extender/SCL: track 201.5 -> 0.00 mm, vias 4 -> 0
- net Net-(J28-Pin_15): track 200.6 -> 0.00 mm, vias 1 -> 0
- net /IO_Extender/SDA: track 187.0 -> 0.00 mm, vias 3 -> 0
- net /Bluetooth/TX: track 180.8 -> 0.00 mm, vias 1 -> 0
- net /UserActions/PB_UP: track 102.3 -> 0.00 mm
- net /UserActions/PB_LEFT: track 100.7 -> 0.00 mm
- net /UserActions/PB_RIGHT: track 95.6 -> 0.00 mm, vias 2 -> 0
- net /UserActions/PB_DOWN: track 83.2 -> 0.00 mm
- net Net-(J26-Pin_2): track 48.6 -> 0.00 mm
- net /LDR: track 47.4 -> 0.00 mm
- net /OLED/A: track 38.9 -> 0.00 mm
- net GND_POWER: track 38.6 -> 0.00 mm, vias 36 -> 0
- net /OLED/B: track 34.7 -> 0.00 mm
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- removed copper zone on B.Cu, net GND
- removed copper zone on F.Cu, net GND
Other:
- board outline removed

Commit message: Add RTC
Parts:
- removed C1, C2: 100nF, Capacitor_SMD:C_0603_1608Metric
- removed J19: Analog_Inputs, Connector_PinHeader_2.54mm:PinHeader_1x04_P2.54mm_Vertical
- removed J20: GND_Analog, Connector_PinHeader_2.54mm:PinHeader_1x04_P2.54mm_Vertical
- removed J21: +3.3V_Analog, Connector_PinHeader_2.54mm:PinHeader_1x04_P2.54mm_Vertical
- removed JP1: J2.54MM, Connector_PinHeader_2.54mm:PinHeader_2x01_P2.54mm_Vertical
- removed R10, R16: 10k, Resistor_THT:R_Axial_DIN0207_L6.3mm_D2.5mm_P7.62mm_Horizontal
- removed SW7: SW_Center, Button_Switch_THT:SW_PUSH_6mm
- removed T1: TestPoint, TestPoint:TestPoint_Pad_1.0x1.0mm
- removed U1: ADS1115IDGS, Package_SO:TSSOP-10_3x3mm_P0.5mm
- added J29: Sig_Servo, Connector_PinHeader_2.54mm:PinHeader_1x01_P2.54mm_Vertical, F.Cu at (113.5, 30.0)
- BT1: footprint Battery:Battery_Panasonic_CR2032-HFN_Horizontal_CircularHoles -> BC501SM:MPD_BC501SM-TR
- J26: value Addr_Selector -> Servo
- R1, R11, R12, R13, R14, R15, R17, R2, R27, R3, R4, R5, R6, R7, R8, R9: footprint Resistor_THT:R_Axial_DIN0207_L6.3mm_D2.5mm_P7.62mm_Horizontal -> Resistor_THT:R_Axial_DIN0207_L6.3mm_D2.5mm_P10.16mm_Horizontal
- moved J2 182.0 mm to (81.3, 29.3), turned to 90 degrees
- moved SW6 166.7 mm to (122.1, 86.1)
- moved U3 164.3 mm to (51.1, 73.2), turned to 180 degrees
- moved H1 162.2 mm to (35.3, 38.1)
- moved BT1 147.7 mm to (66.8, 97.1)
- moved D4 146.6 mm to (52.8, 163.6)
- moved J26 142.2 mm to (113.5, 33.8)
- moved R5 134.9 mm to (56.7, 161.8), turned to 0 degrees
- moved R11 131.3 mm to (83.3, 115.8)
- moved RV1 105.2 mm to (46.2, 84.5)
- moved J13 100.0 mm to (69.5, 76.4)
- moved J15 100.0 mm to (69.5, 81.4)
- moved J36 96.7 mm to (46.0, 105.4), turned to 90 degrees
- moved J16 93.2 mm to (66.4, 39.6)
- moved SW5 76.7 mm to (102.5, 68.6)
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Connections:
- net /IO_Extender/SCL renamed /OLED/SCL
- net /IO_Extender/SDA renamed /OLED/SDA
- J26 pad 3: Net-(J26-Pin_3) -> GND
- J30 pad 2: Net-(J30-Pin_2) -> Net-(J26-Pin_2)
- J32 pad 2: Net-(J30-Pin_2) -> Net-(J26-Pin_2)
- R1 pad 1: +3.3V -> /UserActions/PB_LEFT
- R1 pad 2: /UserActions/PB_LEFT -> GND
- R11 pad 1: +3.3V -> /UserActions/PB_DOWN
- R11 pad 2: /UserActions/PB_DOWN -> GND
- R2 pad 1: +3.3V -> /UserActions/PB_UP
- R2 pad 2: /UserActions/PB_UP -> GND
- R3 pad 1: +3.3V -> /UserActions/PB_RIGHT
- R3 pad 2: /UserActions/PB_RIGHT -> GND
- R4 pad 1: +3.3V -> /UserActions/PB_DOWN
- R4 pad 2: /UserActions/PB_DOWN -> GND
- SW1 pad 1: /UserActions/PB_LEFT -> +3.3V
- SW1 pad 2: GND -> /UserActions/PB_LEFT
- SW2 pad 1: /UserActions/PB_UP -> +3.3V
- SW2 pad 2: GND -> /UserActions/PB_UP
- SW3 pad 1: /UserActions/PB_RIGHT -> +3.3V
- SW3 pad 2: GND -> /UserActions/PB_RIGHT
- SW4 pad 1: /UserActions/PB_DOWN -> +3.3V
- SW4 pad 2: GND -> /UserActions/PB_DOWN
- SW6 pad S1: unconnected-(SW6-PadS1) -> /UserActions/PB_DOWN
- SW6 pad S2: unconnected-(SW6-PadS2) -> +3.3V
- U14 pad 3: unconnected-(U14-VBAT-Pad3) -> Net-(BT1-+)
- U14 pad 8: +3.3V -> /RTC/+5V
Routing:
- net Net-(J5-Pin_8): track 0.00 -> 7.62 mm
- net Net-(J5-Pin_3): track 0.00 -> 7.62 mm
- net Net-(J5-Pin_18): track 0.00 -> 7.62 mm
- net Net-(J5-Pin_13): track 0.00 -> 7.62 mm
- net Net-(J28-Pin_5): track 0.00 -> 7.62 mm
- net Net-(J28-Pin_35): track 0.00 -> 7.62 mm
- net Net-(J28-Pin_15): track 0.00 -> 7.62 mm
Other:
- board outline added: 133.3 x 147.6 mm
- board text added: "+3.3V_EN"
- board text added: "+5V_USB"
- board text added: "3.3V->"
- board text added: "<- Sig Servo_1"
- board text added: "<-5.0V"
- board text added: "<-Power Servo"
- board text added: "ADC_VREF"
- board text added: "AGND"
- board text added: "ANALOG"
- board text added: "BME280 Power selector"
- board text added: "BME280 Temperature Humidity Pressure"
- board text added: "Common"
- board text added: "External"
- board text added: "GP00"
- board text added: "GP01"
- board text added: "GP02"
- board text added: "GP03"
- board text added: "GP04"
- board text added: "GP05"
- board text added: "GP06"
- board text added: "GP07"
- board text added: "GP08"
- board text added: "GP09"
- board text added: "GP10"
- board text added: "GP11"
- board text added: "GP12"
- board text added: "GP13"
- board text added: "GP16"
- board text added: "GP17"
- board text added: "GP18"
- board text added: "GP19"
- board text added: "GP20"
- board text added: "GP21"
- board text added: "GP22"
- board text added: "GP26_A0"
- board text added: "GP27_A1"
- board text added: "GP28_A2"
- board text added: "MPU6050 Accelerometer Gyroscope"
- board text added: "POWER"
- board text added: "RPI_PICO"
- board text added: "RUN"
- board text added: "Servo_1 GND-Vcc-Sig"
- board text added: "Servo_2 GND-Vcc-Sig"
- board text added: "Sig Servo_2 ->"
- board text added: "USB"
- board text added: "VBUS"
- board text added: "VSYS"
- board text removed: "+3.3V ->"
- board text removed: "+5V"
- board text removed: "0x48"
- board text removed: "0x49"
- board text removed: "<- Power Servo Ext-Common-Internal 5V"
- board text removed: "<- Sig Servo"
- board text removed: "A0"
- board text removed: "A1"
- board text removed: "A2"
- board text removed: "A3"
- board text removed: "ADC ->"
- board text removed: "ADC0"
- board text removed: "ADR_1"
- board text removed: "ADR_2"
- board text removed: "Address Selector"
- board text removed: "BME280"
- board text removed: "CLK"
- board text removed: "COMMON"
- board text removed: "CS"
- board text removed: "D1"
- board text removed: "D2"
- board text removed: "D3"
- board text removed: "D4"
- board text removed: "D5"
- board text removed: "D6"
- board text removed: "D7"
- board text removed: "D8"
- board text removed: "EN"
- board text removed: "GND ->"
- board text removed: "GND.+5V.NC"
- board text removed: "Green"
- board text removed: "HC-05 - Bluetooth"
- board text removed: "LED RTC"
- board text removed: "MISO"
- board text removed: "MOSI"
- board text removed: "NC"
- board text removed: "OLED"
- board text removed: "Orange"
- board text removed: "POT"
- board text removed: "Power_Selector"
- board text removed: "RST"
- board text removed: "RX"
- board text removed: "Red"
- board text removed: "Remove D8 Jumper or press Left button when uploading program"
- board text removed: "Servo GND-Vcc-Sig"
- board text removed: "TX"

Commit message: Add codes
Parts:
- added J19: Conn_01x04_Socket, Connector_JST:JST_PH_B4B-PH-K_1x04_P2.00mm_Vertical, F.Cu at (83.3, 165.9)
- added J20: Conn_01x04_Socket, Connector_JST:JST_PH_B4B-PH-K_1x04_P2.00mm_Vertical, F.Cu at (125.0, 149.8)
- added J21: Conn_01x04_Socket, Connector_JST:JST_PH_B4B-PH-K_1x04_P2.00mm_Vertical, F.Cu at (130.7, 149.8)
- moved J10 57.9 mm to (188.9, 119.2)
- moved J12 57.9 mm to (178.7, 119.2)
- moved J8 57.9 mm to (199.0, 119.2)
- moved J9 57.9 mm to (183.8, 119.2)
- moved J11 57.9 mm to (194.0, 119.2)
- moved J28 7.77 mm to (112.6, 108.8)
Routing:
- net Net-(J28-Pin_5): track 7.62 -> 15.4 mm
- net Net-(J28-Pin_15): track 7.62 -> 15.4 mm
- net Net-(J28-Pin_35): track 7.62 -> 15.4 mm
Other:
- board text added: "I2C0_SCL"
- board text added: "I2C0_SDA"
- board text added: "I2C1_SCL"
- board text added: "I2C1_SDA"
- board text added: "SPI0_CSn"
- board text added: "SPI0_RX"
- board text added: "SPI0_SCK"
- board text added: "SPI0_TX"
- board text added: "UART0_RX"
- board text added: "UART0_TX"
- board text added: "UART1_RX"
- board text added: "UART1_TX"

Commit message: Update V2.0 form factor
Parts:
- removed D12: LED, LED_THT:LED_D5.0mm
- removed J37: Sig_MOSFET, Connector_PinHeader_2.54mm:PinHeader_1x01_P2.54mm_Vertical
- removed JP7: Jumper, Connector_PinHeader_2.54mm:PinHeader_1x02_P2.54mm_Vertical
- removed Q1: IRF520, Package_TO_SOT_THT:TO-220-3_Vertical
- removed Q2: 2N7002, Package_TO_SOT_THT:TO-92_Inline
- removed R12, R27: 270, Resistor_THT:R_Axial_DIN0207_L6.3mm_D2.5mm_P10.16mm_Horizontal
- removed R13, R9: 10k, Resistor_THT:R_Axial_DIN0207_L6.3mm_D2.5mm_P10.16mm_Horizontal
- removed R14, R17: 1k, Resistor_THT:R_Axial_DIN0207_L6.3mm_D2.5mm_P10.16mm_Horizontal
- removed U14: DS1307+, Package_DIP:DIP-8_W7.62mm
- added D6: D, Diode_THT:D_A-405_P7.62mm_Horizontal, F.Cu at (50.1, 193.2)
- added D7: D, Diode_THT:D_A-405_P7.62mm_Horizontal, F.Cu at (50.1, 189.0)
- added J31: ST_PH_B4B-PH-K_1x04_P2.00mm, Connector_JST:JST_PH_B4B-PH-K_1x04_P2.00mm_Vertical, F.Cu at (24.1, 171.6)
- added Q3: 2N7002, Package_TO_SOT_THT:TO-92_Inline, F.Cu at (139.9, 208.0)
- added Q4: IRF520, Package_TO_SOT_THT:TO-220-3_Vertical, F.Cu at (128.1, 207.4)
- added R10: 1k, Resistor_THT:R_Axial_DIN0207_L6.3mm_D2.5mm_P10.16mm_Horizontal, F.Cu at (74.1, 205.2)
- added R16: 10k, Resistor_THT:R_Axial_DIN0207_L6.3mm_D2.5mm_P10.16mm_Horizontal, F.Cu at (74.1, 201.2)
- added R18: 270, Resistor_THT:R_Axial_DIN0207_L6.3mm_D2.5mm_P10.16mm_Horizontal, F.Cu at (74.1, 197.1)
- added R19: 1k, Resistor_THT:R_Axial_DIN0207_L6.3mm_D2.5mm_P10.16mm_Horizontal, F.Cu at (74.1, 193.1)
- added R20: 10k, Resistor_THT:R_Axial_DIN0207_L6.3mm_D2.5mm_P10.16mm_Horizontal, F.Cu at (74.1, 189.0)
- added R33: 1k, Resistor_THT:R_Axial_DIN0207_L6.3mm_D2.5mm_P10.16mm_Horizontal, F.Cu at (207.3, 189.3)
- added R34: 1k, Resistor_THT:R_Axial_DIN0207_L6.3mm_D2.5mm_P10.16mm_Horizontal, F.Cu at (180.0, 215.5)
- added R35: 1k, Resistor_THT:R_Axial_DIN0207_L6.3mm_D2.5mm_P10.16mm_Horizontal, F.Cu at (153.0, 188.0)
- added R36: 1k, Resistor_THT:R_Axial_DIN0207_L6.3mm_D2.5mm_P10.16mm_Horizontal, F.Cu at (180.0, 223.6)
- added R37: 1k, Resistor_THT:R_Axial_DIN0207_L6.3mm_D2.5mm_P10.16mm_Horizontal, F.Cu at (153.0, 193.5)
- added R38: 1k, Resistor_THT:R_Axial_DIN0207_L6.3mm_D2.5mm_P10.16mm_Horizontal, F.Cu at (444.6, 203.4)
- added R39: 1k, Resistor_THT:R_Axial_DIN0207_L6.3mm_D2.5mm_P10.16mm_Horizontal, F.Cu at (207.7, 203.9)
- added R40: 1k, Resistor_THT:R_Axial_DIN0207_L6.3mm_D2.5mm_P10.16mm_Horizontal, F.Cu at (180.0, 239.8)
- added SW7: SW_Left, Button_Switch_THT:SW_PUSH_6mm, F.Cu at (60.3, 193.3)
- added SW8: SW_Right, Button_Switch_THT:SW_PUSH_6mm, F.Cu at (193.4, 205.6)
- added U1: PC817, Package_DIP:DIP-4_W7.62mm, F.Cu at (153.6, 209.4)
- added U11: PC817, Package_DIP:DIP-4_W7.62mm, F.Cu at (204.7, 200.1)
- added U12: PC817, Package_DIP:DIP-4_W7.62mm, F.Cu at (166.3, 197.5)
- added U5: 74HC04, Package_DIP:DIP-14_W7.62mm_Socket, F.Cu at (106.9, 188.8)
- added U6: PC817, Package_DIP:DIP-4_W7.62mm, F.Cu at (204.6, 189.2)
- added U7: PC817, Package_DIP:DIP-4_W7.62mm, F.Cu at (166.4, 186.7)
- added V1: ~, CREPP:VIRTUAL_FOOTPRINT, F.Cu at (97.3, 154.1)
- J1: value Screw_Terminal_01x04 -> Screw_Terminal_01x02; footprint TerminalBlock_Phoenix:TerminalBlock_Phoenix_MKDS-1,5-4-5.08_1x04_P5.08mm_Horizontal -> TerminalBlock_Phoenix:TerminalBlock_Phoenix_MKDS-3-2-5.08_1x02_P5.08mm_Horizontal
- J10: value Right_Connector -> Power_Selector; footprint Connector_PinHeader_2.54mm:PinHeader_2x15_P2.54mm_Vertical -> Connector_PinHeader_2.54mm:PinHeader_1x03_P2.54mm_Vertical
- J11: value Right_Connector -> Screw_Terminal_01x02; footprint Connector_PinHeader_2.54mm:PinHeader_2x15_P2.54mm_Vertical -> TerminalBlock_Phoenix:TerminalBlock_Phoenix_MKDS-3-2-5.08_1x02_P5.08mm_Horizontal
- J12: value Right_Connector -> Screw_Terminal_01x04; footprint Connector_PinHeader_2.54mm:PinHeader_2x15_P2.54mm_Vertical -> TerminalBlock_Phoenix:TerminalBlock_Phoenix_MKDS-1,5-4-5.08_1x04_P5.08mm_Horizontal
- J19: value Conn_01x04_Socket -> Screw_Terminal_01x02; footprint Connector_JST:JST_PH_B4B-PH-K_1x04_P2.00mm_Vertical -> TerminalBlock_Phoenix:TerminalBlock_Phoenix_MKDS-3-2-5.08_1x02_P5.08mm_Horizontal
- J20: value Conn_01x04_Socket -> ST_PH_B4B-PH-K_1x04_P2.00mm
- J21: value Conn_01x04_Socket -> Conn_02x04_Odd_Even; footprint Connector_JST:JST_PH_B4B-PH-K_1x04_P2.00mm_Vertical -> Connector_PinHeader_2.54mm:PinHeader_2x04_P2.54mm_Vertical
- J33: footprint TerminalBlock_Phoenix:TerminalBlock_Phoenix_MKDS-1,5-2_1x02_P5.00mm_Horizontal -> TerminalBlock_Phoenix:TerminalBlock_Phoenix_MKDS-3-2-5.08_1x02_P5.08mm_Horizontal
- J8, J9: value Right_Connector -> ST_PH_B4B-PH-K_1x04_P2.00mm; footprint Connector_PinHeader_2.54mm:PinHeader_2x15_P2.54mm_Vertical -> Connector_JST:JST_PH_B4B-PH-K_1x04_P2.00mm_Vertical
- SW5: value SW_Left -> SW_Right
- U2: value PC817 -> L293D; footprint Package_DIP:DIP-4_W7.62mm -> Package_DIP:DIP-16_W7.62mm_Socket
- U4: value RP2040 -> DS1302+; footprint Package_DFN_QFN:QFN-56-1EP_7x7mm_P0.4mm_EP3.2x3.2mm -> Package_DIP:DIP-8_W7.62mm
- moved J26 238.8 mm to (-10.1, 238.1), turned to -90 degrees
- moved J32 231.3 mm to (5.19, 231.6), turned to -90 degrees
- moved J30 227.5 mm to (17.7, 238.2), turned to -90 degrees
- moved J34 223.2 mm to (27.1, 234.0), turned to 180 degrees
- moved J29 220.0 mm to (31.1, 234.0), turned to 180 degrees
- moved H2 212.2 mm to (41.5, 216.0), turned to 180 degrees
- moved J10 202.5 mm to (3.72, 201.2), turned to 90 degrees
- moved J15 201.5 mm to (205.7, 229.9), turned to 0 degrees
- moved J13 200.5 mm to (198.5, 229.9), turned to 0 degrees
- moved J8 200.4 mm to (18.8, 206.8), turned to 180 degrees
- moved J9 196.7 mm to (7.72, 206.8), turned to 180 degrees
- moved J17 191.8 mm to (-20.5, 227.1), turned to 180 degrees
- moved J1 186.9 mm to (171.4, 245.9), turned to -45 degrees
- moved J33 177.2 mm to (108.5, 213.8), turned to 0 degrees
- moved J12 165.6 mm to (14.0, 136.5), turned to -135 degrees
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Connections:
- D5 pad 1: Net-(D5-K) -> /Motors/L239D_Interfaces/5V_Power
- D5 pad 2: Net-(D5-A) -> /Motors/+V_Control
- J1 pad 1: Net-(D5-K) -> Net-(J1-Pin_1)
- J1 pad 2: Net-(D5-K) -> Net-(J1-Pin_2)
- J10 pad 1: unconnected-(J10-Pin_1-Pad1) -> /I2C_Interface/+3.3V
- J10 pad 2: unconnected-(J10-Pin_2-Pad2) -> /I2C_Interface/VCC_Common
- J10 pad 3: unconnected-(J10-Pin_3-Pad3) -> /I2C_Interface/+5V
- J11 pad 1: unconnected-(J11-Pin_1-Pad1) -> Net-(J11-Pin_1)
- J11 pad 2: unconnected-(J11-Pin_2-Pad2) -> Net-(J11-Pin_2)
- J12 pad 1: +3.3V -> Net-(D6-K)
- J12 pad 2: unconnected-(J12-Pin_2-Pad2) -> Net-(D6-K)
- J12 pad 3: +3.3V -> Net-(D6-A)
- J12 pad 4: unconnected-(J12-Pin_4-Pad4) -> /MOSFET/GND_Power
- J19 pad 1: unconnected-(J19-Pin_1-Pad1) -> Net-(J19-Pin_1)
- J19 pad 2: unconnected-(J19-Pin_2-Pad2) -> Net-(J19-Pin_2)
- J21 pad 1: unconnected-(J21-Pin_1-Pad1) -> GND
- J21 pad 2: unconnected-(J21-Pin_2-Pad2) -> GND
- J21 pad 3: unconnected-(J21-Pin_3-Pad3) -> GND
- J21 pad 4: unconnected-(J21-Pin_4-Pad4) -> GND
- J28 pad 1: unconnected-(J28-Pin_1-Pad1) -> Net-(J28-Pin_1)
- J28 pad 10: unconnected-(J28-Pin_10-Pad10) -> /MCU/GP12
- J28 pad 11: unconnected-(J28-Pin_11-Pad11) -> Net-(J28-Pin_11)
- J28 pad 12: unconnected-(J28-Pin_12-Pad12) -> /MCU/GP11
- J28 pad 13: unconnected-(J28-Pin_13-Pad13) -> Net-(J28-Pin_13)
- J28 pad 14: unconnected-(J28-Pin_14-Pad14) -> /MCU/GP10
- J28 pad 16: unconnected-(J28-Pin_16-Pad16) -> /MCU/GND
- J28 pad 17: unconnected-(J28-Pin_17-Pad17) -> Net-(J28-Pin_17)
- J28 pad 18: unconnected-(J28-Pin_18-Pad18) -> /MCU/GP9
- J28 pad 19: unconnected-(J28-Pin_19-Pad19) -> Net-(J28-Pin_19)
- J28 pad 2: unconnected-(J28-Pin_2-Pad2) -> /MCU/GP15
- J28 pad 20: unconnected-(J28-Pin_20-Pad20) -> /MCU/GP8
- J28 pad 21: unconnected-(J28-Pin_21-Pad21) -> Net-(J28-Pin_21)
- J28 pad 22: unconnected-(J28-Pin_22-Pad22) -> /MCU/GP7
- J28 pad 23: unconnected-(J28-Pin_23-Pad23) -> Net-(J28-Pin_23)
- J28 pad 24: unconnected-(J28-Pin_24-Pad24) -> /MCU/GP6
- J28 pad 25: unconnected-(J28-Pin_25-Pad25) -> Net-(J28-Pin_25)
- J28 pad 26: unconnected-(J28-Pin_26-Pad26) -> /MCU/GND
- J28 pad 27: unconnected-(J28-Pin_27-Pad27) -> Net-(J28-Pin_27)
- J28 pad 28: unconnected-(J28-Pin_28-Pad28) -> /MCU/GP5
- J28 pad 29: unconnected-(J28-Pin_29-Pad29) -> Net-(J28-Pin_29)
- J28 pad 3: unconnected-(J28-Pin_3-Pad3) -> Net-(J28-Pin_3)
- J28 pad 30: unconnected-(J28-Pin_30-Pad30) -> /MCU/GP4
- J28 pad 31: unconnected-(J28-Pin_31-Pad31) -> Net-(J28-Pin_31)
- J28 pad 32: unconnected-(J28-Pin_32-Pad32) -> /MCU/GP3
- J28 pad 33: unconnected-(J28-Pin_33-Pad33) -> Net-(J28-Pin_33)
- J28 pad 34: unconnected-(J28-Pin_34-Pad34) -> /MCU/GP2
- J28 pad 36: unconnected-(J28-Pin_36-Pad36) -> /MCU/GND
- J28 pad 37: unconnected-(J28-Pin_37-Pad37) -> Net-(J28-Pin_37)
- J28 pad 38: unconnected-(J28-Pin_38-Pad38) -> /MCU/GP1
- J28 pad 39: unconnected-(J28-Pin_39-Pad39) -> Net-(J28-Pin_39)
- J28 pad 4: unconnected-(J28-Pin_4-Pad4) -> /MCU/GP14
- J28 pad 40: unconnected-(J28-Pin_40-Pad40) -> /MCU/GP0
- J28 pad 6: unconnected-(J28-Pin_6-Pad6) -> /MCU/GND
- J28 pad 7: unconnected-(J28-Pin_7-Pad7) -> Net-(J28-Pin_7)
- J28 pad 8: unconnected-(J28-Pin_8-Pad8) -> /MCU/GP13
- J28 pad 9: unconnected-(J28-Pin_9-Pad9) -> Net-(J28-Pin_9)
- J4 pad 1: unconnected-(J4-Pin_1-Pad1) -> Net-(J28-Pin_1)
- J4 pad 10: unconnected-(J4-Pin_10-Pad10) -> Net-(J28-Pin_19)
- J4 pad 11: unconnected-(J4-Pin_11-Pad11) -> Net-(J28-Pin_21)
- J4 pad 12: unconnected-(J4-Pin_12-Pad12) -> Net-(J28-Pin_23)
- J4 pad 13: unconnected-(J4-Pin_13-Pad13) -> Net-(J28-Pin_25)
- J4 pad 14: unconnected-(J4-Pin_14-Pad14) -> Net-(J28-Pin_27)
- J4 pad 15: unconnected-(J4-Pin_15-Pad15) -> Net-(J28-Pin_29)
- J4 pad 16: unconnected-(J4-Pin_16-Pad16) -> Net-(J28-Pin_31)
- J4 pad 17: unconnected-(J4-Pin_17-Pad17) -> Net-(J28-Pin_33)
- J4 pad 19: unconnected-(J4-Pin_19-Pad19) -> Net-(J28-Pin_37)
- J4 pad 2: unconnected-(J4-Pin_2-Pad2) -> Net-(J28-Pin_3)
- J4 pad 20: unconnected-(J4-Pin_20-Pad20) -> Net-(J28-Pin_39)
- J4 pad 4: unconnected-(J4-Pin_4-Pad4) -> Net-(J28-Pin_7)
- J4 pad 5: unconnected-(J4-Pin_5-Pad5) -> Net-(J28-Pin_9)
- J4 pad 6: unconnected-(J4-Pin_6-Pad6) -> Net-(J28-Pin_11)
- J4 pad 7: unconnected-(J4-Pin_7-Pad7) -> Net-(J28-Pin_13)
- J4 pad 9: unconnected-(J4-Pin_9-Pad9) -> Net-(J28-Pin_17)
- J5 pad 10: unconnected-(J5-Pin_10-Pad10) -> Net-(J5-Pin_10)
- J5 pad 11: unconnected-(J5-Pin_11-Pad11) -> Net-(J5-Pin_11)
- J5 pad 12: unconnected-(J5-Pin_12-Pad12) -> Net-(J5-Pin_12)
- J5 pad 14: unconnected-(J5-Pin_14-Pad14) -> Net-(J5-Pin_14)
- J5 pad 15: unconnected-(J5-Pin_15-Pad15) -> Net-(J5-Pin_15)
- J5 pad 16: unconnected-(J5-Pin_16-Pad16) -> Net-(J5-Pin_16)
- J5 pad 17: unconnected-(J5-Pin_17-Pad17) -> Net-(J5-Pin_17)
- J5 pad 19: unconnected-(J5-Pin_19-Pad19) -> Net-(J5-Pin_19)
- J5 pad 20: unconnected-(J5-Pin_20-Pad20) -> Net-(J5-Pin_20)
- J5 pad 7: unconnected-(J5-Pin_7-Pad7) -> Net-(J5-Pin_7)
- J5 pad 9: unconnected-(J5-Pin_9-Pad9) -> Net-(J5-Pin_9)
- J6 pad 13: unconnected-(J6-Pin_13-Pad13) -> Net-(J5-Pin_7)
- J6 pad 17: unconnected-(J6-Pin_17-Pad17) -> Net-(J5-Pin_9)
- J6 pad 19: unconnected-(J6-Pin_19-Pad19) -> Net-(J5-Pin_10)
- J6 pad 21: unconnected-(J6-Pin_21-Pad21) -> Net-(J5-Pin_11)
- J6 pad 23: unconnected-(J6-Pin_23-Pad23) -> Net-(J5-Pin_12)
- J6 pad 27: unconnected-(J6-Pin_27-Pad27) -> Net-(J5-Pin_14)
- J6 pad 29: unconnected-(J6-Pin_29-Pad29) -> Net-(J5-Pin_15)
- J6 pad 31: unconnected-(J6-Pin_31-Pad31) -> Net-(J5-Pin_16)
- J6 pad 32: unconnected-(J6-Pin_32-Pad32) -> /MCU/GP19
- J6 pad 33: unconnected-(J6-Pin_33-Pad33) -> Net-(J5-Pin_17)
- J6 pad 34: unconnected-(J6-Pin_34-Pad34) -> /MCU/GP18
- J6 pad 37: unconnected-(J6-Pin_37-Pad37) -> Net-(J5-Pin_19)
- J6 pad 39: unconnected-(J6-Pin_39-Pad39) -> Net-(J5-Pin_20)
- J6 pad 40: unconnected-(J6-Pin_40-Pad40) -> /MCU/GP16
- J8 pad 1: unconnected-(J8-Pin_1-Pad1) -> /I2C_Interface/VCC_Common
- J8 pad 2: GND -> /I2C_Interface/SCL
- J8 pad 3: unconnected-(J8-Pin_3-Pad3) -> /I2C_Interface/SDA
- J8 pad 4: GND -> /I2C_Interface/GND
- J9 pad 1: unconnected-(J9-Pin_1-Pad1) -> /I2C_Interface/VCC_Common
- J9 pad 2: unconnected-(J9-Pin_2-Pad2) -> /I2C_Interface/SCL
- J9 pad 3: unconnected-(J9-Pin_3-Pad3) -> /I2C_Interface/SDA
- J9 pad 4: unconnected-(J9-Pin_4-Pad4) -> /I2C_Interface/GND
- SW5 pad 2: Net-(R17-Pad1) -> /Motors/L239D_Interfaces/GND
- U2 pad 1: Net-(Q2-D) -> /Motors/L239D_Interfaces/EN_M1_OUT
- U2 pad 2: GND -> /Motors/L239D_Interfaces/DIR_M1_A
- U2 pad 3: GND_POWER -> Net-(J1-Pin_1)
- U2 pad 4: Net-(Q1-G) -> /Motors/GND_Power
- U3 pad 1: unconnected-(U3-GND-Pad1) -> /NRF24/GND
- U3 pad 2: unconnected-(U3-VCC-Pad2) -> /NRF24/+3.3V
- U3 pad 3: unconnected-(U3-CE-Pad3) -> /NRF24/CE
- U3 pad 4: unconnected-(U3-~{CSN}-Pad4) -> /NRF24/~{CSN}
- U3 pad 5: unconnected-(U3-SCK-Pad5) -> /NRF24/SCK
- U3 pad 6: unconnected-(U3-MOSI-Pad6) -> /NRF24/MOSI
- U3 pad 7: unconnected-(U3-MISO-Pad7) -> /NRF24/MISO
- U4 pad 1: Net-(U4-IOVDD-Pad1) -> +3.3V
- U4 pad 2: unconnected-(U4-GPIO0-Pad2) -> Net-(U4-X1)
- U4 pad 3: unconnected-(U4-GPIO1-Pad3) -> Net-(U4-X2)
- U4 pad 4: unconnected-(U4-GPIO2-Pad4) -> GND
- U4 pad 5: unconnected-(U4-GPIO3-Pad5) -> /RTC/CE
- U4 pad 6: unconnected-(U4-GPIO4-Pad6) -> /RTC/MOSI
- U4 pad 7: unconnected-(U4-GPIO5-Pad7) -> /RTC/SCK
- U4 pad 8: unconnected-(U4-GPIO6-Pad8) -> Net-(BT1-+)
- Y2 pad 1: Net-(U14-X1) -> Net-(U4-X1)
- Y2 pad 2: Net-(U14-X2) -> Net-(U4-X2)
Routing:
- net /MOSFET/GND_Power: track 0.00 -> 29.2 mm
- net Net-(J28-Pin_39): track 0.00 -> 15.4 mm
- net Net-(J28-Pin_33): track 0.00 -> 15.4 mm
- net Net-(J28-Pin_29): track 0.00 -> 15.4 mm
- net Net-(J28-Pin_27): track 0.00 -> 15.4 mm
- net Net-(J28-Pin_21): track 0.00 -> 15.4 mm
- net Net-(J28-Pin_19): track 0.00 -> 15.4 mm
- net Net-(J28-Pin_17): track 0.00 -> 15.4 mm
- net Net-(J28-Pin_13): track 0.00 -> 15.4 mm
- net Net-(J28-Pin_37): track 0.00 -> 15.4 mm
- net Net-(J28-Pin_31): track 0.00 -> 15.4 mm
- net Net-(J28-Pin_23): track 0.00 -> 15.4 mm
- net Net-(J28-Pin_35): track 15.4 -> 0.03 mm
- net Net-(D6-K): track 0.00 -> 14.3 mm
- net Net-(D6-A): track 0.00 -> 10.3 mm
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- removed copper zone on B.Cu, net GND_POWER
- removed copper zone on F.Cu, net GND_POWER
Other:
- board size 133.3 x 147.6 mm -> 247.5 x 183.2 mm
- board text added: "+5V"
- board text added: "GND.SDA.SCL.VCC"
- board text added: "GP14"
- board text added: "GP15"
- board text added: "I2C Voltage selection"
- board text added: "I2C0"
- board text added: "NFR24_TRANSCEIVER"
- board text removed: "+5V_USB"
- board text removed: "<- Sig Servo_1"
- board text removed: "<-Power Servo"
- board text removed: "Common"
- board text removed: "D0"
- board text removed: "External"
- board text removed: "GND_2"
- board text removed: "LDR"
- board text removed: "LOAD+"
- board text removed: "LOAD-"
- board text removed: "MOSFET"
- board text removed: "POWERED"
- board text removed: "Servo_1 GND-Vcc-Sig"
- board text removed: "Servo_2 GND-Vcc-Sig"
- board text removed: "Sig MOSFET"
- board text removed: "Sig Servo_2 ->"
- board text removed: "VCC GND"

Commit message: Add img
Parts:
- added H5: MountingHole, MountingHole:MountingHole_2.1mm, F.Cu at (174.3, 78.2)
- added H6: MountingHole, MountingHole:MountingHole_2.1mm, F.Cu at (174.5, 51.2)
- added JP1: Jumper_2.54mm_red, CREPP_Jumpers:Jumper_2.54mm_red, F.Cu at (154.2, 123.4)
- added JP10: Jumper_2.54mm_green, CREPP_Jumpers:Jumper_2.54mm_green, F.Cu at (197.6, 126.0)
- added JP11: Jumper_2.54mm_green, CREPP_Jumpers:Jumper_2.54mm_green, F.Cu at (197.6, 131.1)
- added JP12: Jumper_2.54mm_green, CREPP_Jumpers:Jumper_2.54mm_green, F.Cu at (197.6, 120.9)
- added JP13: Jumper_2.54mm_green, CREPP_Jumpers:Jumper_2.54mm_green, F.Cu at (197.6, 108.2)
- added JP14: Jumper_2.54mm_green, CREPP_Jumpers:Jumper_2.54mm_green, F.Cu at (197.6, 98.0)
- added JP15: Jumper_2.54mm_green, CREPP_Jumpers:Jumper_2.54mm_green, F.Cu at (197.6, 93.0)
- added JP16: Jumper_2.54mm_green, CREPP_Jumpers:Jumper_2.54mm_green, F.Cu at (197.6, 133.6)
- added JP17: Jumper_2.54mm_green, CREPP_Jumpers:Jumper_2.54mm_green, F.Cu at (197.6, 87.9)
- added JP18: Jumper_2.54mm_green, CREPP_Jumpers:Jumper_2.54mm_green, F.Cu at (197.6, 113.3)
- added JP19: Jumper_2.54mm_green, CREPP_Jumpers:Jumper_2.54mm_green, F.Cu at (197.6, 123.4)
- added JP2: Jumper_2.54mm_red, CREPP_Jumpers:Jumper_2.54mm_red, F.Cu at (154.2, 131.1)
- added JP20: Jumper_2.54mm_green, CREPP_Jumpers:Jumper_2.54mm_green, F.Cu at (154.2, 118.4)
- added JP21: Jumper_2.54mm_green, CREPP_Jumpers:Jumper_2.54mm_green, F.Cu at (154.2, 113.3)
- added JP22: Jumper_2.54mm_green, CREPP_Jumpers:Jumper_2.54mm_green, F.Cu at (154.2, 110.7)
- added JP23: Jumper_2.54mm_green, CREPP_Jumpers:Jumper_2.54mm_green, F.Cu at (154.2, 105.7)
- added JP24: Jumper_2.54mm_green, CREPP_Jumpers:Jumper_2.54mm_green, F.Cu at (154.2, 100.6)
- added JP25: Jumper_2.54mm_green, CREPP_Jumpers:Jumper_2.54mm_green, F.Cu at (154.2, 98.0)
- added JP26: Jumper_2.54mm_green, CREPP_Jumpers:Jumper_2.54mm_green, F.Cu at (154.2, 95.5)
- added JP27: Jumper_2.54mm_green, CREPP_Jumpers:Jumper_2.54mm_green, F.Cu at (154.2, 93.0)
- added JP28: Jumper_2.54mm_green, CREPP_Jumpers:Jumper_2.54mm_green, F.Cu at (154.2, 87.9)
- added JP29: Jumper_2.54mm_green, CREPP_Jumpers:Jumper_2.54mm_green, F.Cu at (154.2, 85.3)
- added JP3: Jumper_2.54mm_red, CREPP_Jumpers:Jumper_2.54mm_red, F.Cu at (154.2, 133.6)
- added JP4: Jumper_2.54mm_green, CREPP_Jumpers:Jumper_2.54mm_green, F.Cu at (197.6, 85.3)
- added JP5: Jumper_2.54mm_green, CREPP_Jumpers:Jumper_2.54mm_green, F.Cu at (197.6, 110.7)
- added JP6: Jumper_2.54mm_green, CREPP_Jumpers:Jumper_2.54mm_green, F.Cu at (197.6, 118.4)
- added JP7: Jumper_2.54mm_green, CREPP_Jumpers:Jumper_2.54mm_green, F.Cu at (197.6, 105.7)
- added JP8: Jumper_2.54mm_green, CREPP_Jumpers:Jumper_2.54mm_green, F.Cu at (197.6, 100.6)
- added JP9: Jumper_2.54mm_green, CREPP_Jumpers:Jumper_2.54mm_green, F.Cu at (197.6, 95.5)
- added M1: Motor_DC, Connector_PinHeader_2.54mm:PinHeader_1x01_P2.54mm_Vertical, B.Cu at (285.8, 175.2)
- added M2: Motor_DC, Connector_PinHeader_2.54mm:PinHeader_1x01_P2.54mm_Vertical, B.Cu at (64.8, 175.2)
- added M3: Motor_DC, Connector_PinHeader_2.54mm:PinHeader_1x01_P2.54mm_Vertical, F.Cu at (293.5, 107.3)
- added S1: ~, CREPP_Spacers:Spacer_M3_FF_20mm, F.Cu at (232.3, 69.7)
- added S2: ~, CREPP_Spacers:Spacer_M3_FF_20mm, F.Cu at (232.8, 172.2)
- added S3: ~, CREPP_Spacers:Spacer_M3_FF_20mm, F.Cu at (117.3, 172.2)
- added S4: ~, CREPP_Spacers:Spacer_M3_FF_20mm, F.Cu at (117.3, 69.7)
- added SERVO_SG1: ~, CREPP_Servo:SG90_Servo, F.Cu at (174.4, 56.9)
- U1, U11, U12, U6, U7: footprint Package_DIP:DIP-4_W7.62mm -> Package_DIP:SMDIP-4_W9.53mm
- moved R38 207.4 mm to (240.3, 167.7)
- moved BT1 120.1 mm to (216.3, 136.2)
- moved J27 115.1 mm to (208.9, 81.4)
- moved J23 115.1 mm to (206.3, 76.6)
- moved Q4 93.9 mm to (201.3, 148.7)
- moved SW7 93.2 mm to (150.6, 169.9)
- moved J33 89.1 mm to (184.3, 167.0)
- moved U5 88.9 mm to (182.5, 142.0)
- moved J19 88.7 mm to (156.7, 167.0)
- moved U2 88.5 mm to (155.7, 140.8)
- moved J2 87.9 mm to (178.8, 59.7)
- moved D2 87.6 mm to (85.7, 133.3)
- moved R10 87.6 mm to (149.9, 161.4)
- moved R18 87.6 mm to (149.9, 153.3)
- moved SW3 87.6 mm to (242.6, 111.9)
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Connections:
- J19 pad 2: Net-(J19-Pin_2) -> unconnected-(J19-Pin_2-Pad2)
- U2 pad 16: Net-(J19-Pin_2) -> Net-(J19-Pin_1)
Routing:
- net /MOSFET/GND_Power: track 29.2 -> 22.9 mm
- net /Motors/L239D_Interfaces/GND: track 0.00 -> 6.33 mm
Other:
- outline, holes or cut-outs redrawn
- board text added: "Enable Motor_1"
- board text added: "Enable Motor_2"
- board text added: "Motor_1"
- board text added: "Motor_2"
- board text added: "SERVOMOTOR"
- board text added: "V_{MOTOR}.GND"
- board text added: "V_{SERVO}.GND"
- board text removed: "Power_Servo"
