File: PCB/V2.0/CREPP.io.kicad_pcb (KiCad board)
At the start: 2 copper layers, 247.5 x 183.2 mm, 131 parts, among them J1 Screw_Terminal_01x02, J11 Screw_Terminal_01x02, J12 Screw_Terminal_01x04, J13 Conn_02x04_Odd_Even, J14 OLED_SOCKET, J15 Conn_02x04_Odd_Even, J16 I2C_Selector, J17 Conn_02x04_Odd_Even, J18 Conn_02x04_Odd_Even, J19 Screw_Terminal_01x02, J2 HC-SR04_VIRTUAL, J21 Conn_02x04_Odd_Even, J23 HC-SR, J25 BME, J26 Servo, J27 SIG_HCSR04, J28 Conn_02x20, J29 Sig_Servo, J3 Conn_02x04_Odd_Even, J30 Servo, J32 Power_Servo_Selector, J33 Screw_Terminal_01x02, J34 Sig_Servo, J36 Power_Selector, J4 Conn_01x20, J40 Conn_01x08_Socket, J5 Conn_01x20, J6 Conn_02x20, J7 VIRTUAL_MPU6050, J8 Coon_01x04_Pin_2mm, J9 Coon_01x04_Pin_2mm, M1 Motor_DC, M2 Motor_DC, Q3 2N7002, Q4 IRF520, SW1 SW_Left, SW2 SW_Up, SW3 SW_Right, SW4 SW_Down, SW5 SW_Right, SW6 RotaryEncoder_Switch, SW7 SW_Left, SW8 SW_Right, SW9 SW_Left, U1 PC817_SMD, U2 L293D, U3 NRF24L01_Breakout, U4 DS3231M, U5 74HC04, U6 PC817_SMD, U7 PC817_SMD, U8 PC817_SMD, U9 PC817_SMD

Commit message: Update
Parts:
- removed J27: SIG_HCSR04, Connector_PinHeader_2.54mm:PinHeader_1x02_P2.54mm_Vertical
- removed J9: Coon_01x04_Pin_2mm, Connector_JST:JST_PH_B4B-PH-K_1x04_P2.00mm_Vertical
- added D10: LED_Green, CREPP_LEDs:LED_D5.0mm_Green, F.Cu at (282.6, 119.9)
- added D11: LED_Orange, CREPP_LEDs:LED_D5.0mm_Orange, F.Cu at (275.5, 107.2)
- added D12: LED, LED_THT:LED_D5.0mm, F.Cu at (95.1, 135.3)
- added D13: LED, LED_THT:LED_D5.0mm, F.Cu at (94.3, 146.8)
- added D9: LED_Red, CREPP_LEDs:LED_D5.0mm_Red, F.Cu at (267.1, 95.5)
- added J35: HC-SR04_VIRTUAL, Connector_PinSocket_2.54mm:PinSocket_1x04_P2.54mm_Vertical, F.Cu at (278.7, 53.8)
- added J37: Servo, Connector_PinHeader_2.54mm:PinHeader_1x03_P2.54mm_Vertical, F.Cu at (191.0, 73.7)
- added R12: 270, Resistor_THT:R_Axial_DIN0207_L6.3mm_D2.5mm_P10.16mm_Horizontal, F.Cu at (262.8, 127.1)
- added R13: 270, Resistor_THT:R_Axial_DIN0207_L6.3mm_D2.5mm_P10.16mm_Horizontal, F.Cu at (270.9, 138.3)
- added R14: 270, Resistor_THT:R_Axial_DIN0207_L6.3mm_D2.5mm_P10.16mm_Horizontal, F.Cu at (268.9, 135.3)
- added R17: 270, Resistor_THT:R_Axial_DIN0207_L6.3mm_D2.5mm_P10.16mm_Horizontal, F.Cu at (84.8, 129.5)
- added R21: 270, Resistor_THT:R_Axial_DIN0207_L6.3mm_D2.5mm_P10.16mm_Horizontal, F.Cu at (84.0, 141.0)
- added U11: ~, CREPP_NRF24:nRF24L01_Virtual, F.Cu at (142.8, 80.6)
- added U12: PCA9635, Package_SO:TSSOP-28_4.4x9.7mm_P0.65mm, F.Cu at (214.6, 137.8)
- added U13: ST890, CREPP_PMOS_CMS:ST890, F.Cu at (84.7, 136.3)
- added U14: ST890, CREPP_PMOS_CMS:ST890, F.Cu at (84.7, 144.9)
- D1: value LED -> LED_Red; footprint LED_THT:LED_D5.0mm -> CREPP_LEDs:LED_D5.0mm_Red
- D2: value LED -> LED_Orange; footprint LED_THT:LED_D5.0mm -> CREPP_LEDs:LED_D5.0mm_Orange
- D3, D4: value LED -> LED_Green; footprint LED_THT:LED_D5.0mm -> CREPP_LEDs:LED_D5.0mm_Green
- J2: value HC-SR04_VIRTUAL -> Coon_01x04_Pin_2mm; footprint Connector_PinSocket_2.54mm:PinSocket_1x04_P2.54mm_Vertical -> Connector_JST:JST_PH_B4B-PH-K_1x04_P2.00mm_Vertical
- J23: value HC-SR -> Coon_01x04_Pin_2mm; footprint Connector_PinSocket_2.54mm:PinSocket_1x04_P2.54mm_Vertical -> Connector_JST:JST_PH_B4B-PH-K_1x04_P2.00mm_Vertical
- JP8, JP9: value Jumper_2.54mm_green -> Jumper_2.54mm_blue; footprint CREPP_Jumpers:Jumper_2.54mm_green -> CREPP_Jumpers:Jumper_2.54mm_blue
- SW9: value SW_Left -> SW_Reset
- U3: value NRF24L01_Breakout -> NRF24L01_Breakout_socket; footprint RF_Module:nRF24L01_Breakout -> CREPP_NRF24:nRF24L01_Breakout
- moved OLED1 199.5 mm to (114.4, 83.6)
- moved D1 195.2 mm to (271.5, 101.3), turned to -145 degrees
- moved D2 194.5 mm to (279.1, 113.5), turned to -150 degrees
- moved RV1 183.3 mm to (73.6, 109.8), turned to -30 degrees
- moved R7 174.9 mm to (264.9, 129.9), turned to 60 degrees
- moved G*** 173.8 mm to (215.5, 67.3)
- moved R6 173.4 mm to (266.8, 132.6), turned to 60 degrees
- moved J8 160.7 mm to (248.4, 116.0), turned to -90 degrees
- moved R8 127.5 mm to (200.4, 81.7), turned to 90 degrees
- moved D3 127.4 mm to (200.4, 65.8)
- moved J2 96.6 mm to (257.2, 116.1)
- moved SW9 92.1 mm to (126.8, 136.5), turned to 90 degrees
- moved J14 91.7 mm to (118.2, 83.6)
- moved D4 87.6 mm to (135.4, 131.7), turned to 0 degrees
- moved LDR1 85.9 mm to (129.0, 117.4), turned to 0 degrees
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Connections:
- D4 pad 1: Net-(D4-K) -> GND
- D4 pad 2: +5V -> Net-(D4-A)
- J13 pad 2: /I2C_Interface/SCL -> /SCL
- J13 pad 4: /I2C_Interface/SCL -> /SCL
- J13 pad 6: /I2C_Interface/SCL -> /SCL
- J13 pad 8: /I2C_Interface/SCL -> /SCL
- J15 pad 1: /I2C_Interface/SDA -> /SDA
- J15 pad 2: +3.3V -> /MCU/+3.3V
- J15 pad 3: /I2C_Interface/SDA -> /SDA
- J15 pad 4: +3.3V -> /MCU/+3.3V
- J15 pad 5: /I2C_Interface/SDA -> /SDA
- J15 pad 6: +3.3V -> /MCU/+3.3V
- J15 pad 7: /I2C_Interface/SDA -> /SDA
- J15 pad 8: +3.3V -> /MCU/+3.3V
- J16 pad 1: /I2C_Interface/SDA -> /SDA
- J16 pad 2: /I2C_Interface/SDA -> /SDA
- J16 pad 5: /I2C_Interface/SCL -> /SCL
- J16 pad 6: /I2C_Interface/SCL -> /SCL
- J2 pad 1: unconnected-(J2-Pin_1-Pad1) -> GND
- J2 pad 2: unconnected-(J2-Pin_2-Pad2) -> /SDA
- J2 pad 3: unconnected-(J2-Pin_3-Pad3) -> /SCL
- J2 pad 4: unconnected-(J2-Pin_4-Pad4) -> +3.3V
- J23 pad 1: GND -> /HC-SR04/+3.3V
- J23 pad 2: Net-(J23-Pin_2) -> /HC-SR04/TRIG
- J23 pad 3: Net-(J23-Pin_3) -> /HC-SR04/ECHO
- J23 pad 4: +3.3V -> /HC-SR04/GND
- J25 pad 3: /I2C_Interface/SDA -> /SDA
- J25 pad 4: /I2C_Interface/SCL -> /SCL
- J28 pad 2: /MCU/GP15 -> /HC-SR04/TRIG
- J28 pad 20: /LED/GREEN -> /MCU/GP8
- J28 pad 22: /LED/ORANGE_LED -> /MCU/GP7
- J28 pad 24: /LED/RED_LED -> /MCU/GP6
- J28 pad 28: /I2C_Interface/SCL -> /SCL
- J28 pad 30: /I2C_Interface/SDA -> /SDA
- J28 pad 4: /MCU/GP14 -> /HC-SR04/ECHO
- J28 pad 8: /MCU/GP13 -> /DEFAULT_LED
- J40 pad 3: /I2C_Interface/SDA -> /SDA
- J40 pad 4: /I2C_Interface/SCL -> /SCL
- J6 pad 10: +3.3V -> /MCU/+3.3V
- J6 pad 14: unconnected-(J6-Pin_14-Pad14) -> /MCU/GP28
- J6 pad 18: unconnected-(J6-Pin_18-Pad18) -> /MCU/GP27
- J6 pad 2: +5V -> /Power_Supply1/IN
- J6 pad 20: unconnected-(J6-Pin_20-Pad20) -> /MCU/GP26
- J6 pad 36: unconnected-(J6-Pin_36-Pad36) -> /MCU/GND
- J6 pad 38: unconnected-(J6-Pin_38-Pad38) -> /MCU/GP17
- J8 pad 2: /I2C_Interface/SDA -> /SDA
- J8 pad 3: /I2C_Interface/SCL -> /SCL
- R11 pad 1: /MCU/GP13 -> /MCU/GP8
- R5 pad 1: Net-(D4-K) -> +5V
- R5 pad 2: GND -> Net-(D4-A)
- R6 pad 1: /LED/RED_LED -> /IO_Extender/LED_3
- R6 pad 2: Net-(D1-A) -> Net-(D11-A)
- R7 pad 1: /LED/ORANGE_LED -> /IO_Extender/LED_4
- R7 pad 2: Net-(D2-A) -> Net-(D1-A)
- R8 pad 1: /LED/GREEN -> /DEFAULT_LED
- R9 pad 2: GND -> +3.3V
- SW6 pad A: /MCU/GP14 -> /MCU/GP7
- SW6 pad B: /MCU/GP15 -> /MCU/GP6
- SW6 pad S1: /MCU/GP13 -> /MCU/GP8
- U3 pad 3: /MCU/GP21 -> /MCU/GP20
- U3 pad 4: /MCU/GP20 -> /MCU/GP21
- U4 pad 15: /I2C_Interface/SDA -> /SDA
- U4 pad 16: /I2C_Interface/SCL -> /SCL
Routing:
- net +3.3V: track 0.00 -> 138.0 mm
- net /SDA: track 0.00 -> 65.6 mm, vias 0 -> 4
- net /SCL: track 0.00 -> 63.1 mm, vias 0 -> 2
- net /IO_Extender/LED_1: track 0.00 -> 54.1 mm
- net /IO_Extender/LED_2: track 0.00 -> 51.8 mm
- net /IO_Extender/LED_3: track 0.00 -> 50.6 mm
- net /IO_Extender/LED_4: track 0.00 -> 49.4 mm
- net /IO_Extender/LED_5: track 0.00 -> 48.2 mm
- net /OLED/B: track 0.00 -> 30.8 mm
- net /MCU/GP27: track 0.00 -> 25.1 mm
- net /MCU/RUN: track 0.00 -> 24.4 mm
- net Net-(D9-A): track 0.00 -> 22.3 mm
- net Net-(BT1-+): track 0.00 -> 20.3 mm, vias 0 -> 2
- net Net-(D1-A): track 0.00 -> 18.6 mm
- net Net-(D4-A): track 0.00 -> 18.2 mm
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Other:
- board text added: "3.3V.SCL.SDA.GND"
- board text added: "CREPP.io V2.0 - 2024"
- board text added: "GND.Sig.VCC"
- board text added: "NRF24"
- board text added: "Power_OK"
- board text added: "RESET"
- board text added: "Reset"
- board text removed: "3.3V->"
- board text removed: "<-5.0V"
- board text removed: "A"
- board text removed: "B"
- board text removed: "BME280 Power selector"
- board text removed: "GND-3.3V-B-A"
- board text removed: "GND.SDA.SCL.VCC"
- board text removed: "HCSR-04"
- board text removed: "I2C Voltage selection"
