File: PCB/V2.0/Modules/L239D_Interfaces.kicad_sch (KiCad schematic)
At the start: 15 parts, among them SW5 SW_Right, SW8 SW_Right, U11 PC817, U12 PC817, U5 74HC04, U6 PC817, U7 PC817

Commit message: Add img
Parts:
- removed U11, U12, U6, U7: PC817, Package_DIP:DIP-4_W7.62mm, symbol Isolator:PC817
- added U6, U7, U8, U9: PC817_SMD, Package_DIP:SMDIP-4_W9.53mm, symbol CREPP_Optocoupler:PC817_SMD
Connections:
- net DIR_M1_B: now also U6.4
- net DIR_M2_B: now also U8.4
- net GND_Logic: now also U6.2, U6.3, U7.2, U7.3, U8.2, U8.3, U9.2, U9.3
- net at R39.1: now also U8.1
- net at R37.1: now also U9.1
- net at R35.1: now also U7.1
- net at R36.1, SW8.1, U5.5: now also U7.4
- net at R33.1: now also U6.1
- net at R38.1, SW5.1, U5.9: now also U9.4
