File: PCB/V2.0/Modules/Motors.kicad_sch (KiCad schematic)
At the start: 5 parts, among them J1 Screw_Terminal_01x02, J11 Screw_Terminal_01x02, J19 Screw_Terminal_01x02, U2 L293D

Commit message: Add img
Parts:
- removed U2: L293D, Package_DIP:DIP-16_W7.62mm_Socket, symbol Driver_Motor:L293D
- added M1, M2: Motor_DC, Connector_PinHeader_2.54mm:PinHeader_1x01_P2.54mm_Vertical, symbol Motor:Motor_DC
- added U2: L293D, Package_DIP:DIP-16_W7.62mm_Socket, symbol CREPP_Drivers_Motors:L293D_THT
Connections:
- net GND_Power: now also U2.12 (GND), U2.13 (GND), U2.4 (GND), U2.5 (GND)
- net L239D_Interfaces/DIR_M1_A: now also U2.2 (1A)
- net L239D_Interfaces/DIR_M1_B: now also U2.7 (2A)
- net L239D_Interfaces/DIR_M2_A: now also U2.10 (3A)
- net L239D_Interfaces/DIR_M2_B: now also U2.15 (4A)
- net L239D_Interfaces/EN_M1_OUT: now also U2.1 (EN1,2)
- net L239D_Interfaces/EN_M2_OUT: now also U2.9 (EN3,4)
- net at J1.1 (Pin_1): now also U2.3 (1Y)
- net at J1.2 (Pin_2): now also U2.6 (2Y)
- net at J11.1 (Pin_1): now also U2.11 (3Y)
- net at J11.2 (Pin_2): now also U2.14 (4Y)
- net at J19.1 (Pin_1): now also U2.16 (VCC1), U2.8 (VCC2)
Changed lines of the file:
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@@
+	)
+	(junction
+		(at 152.4 60.96)
+		(diameter 0)
+		(color 0 0 0 0)
 	)
 	(junction
@@
 	(wire
 		(pts
+			(xy 152.4 53.34) (xy 152.4 60.96)
+		)
+		(stroke
+			(width 0)
+			(type default)
+		)
+	)
+	(wire
+		(pts
 			(xy 78.74 80.01) (xy 92.71 80.01)
 		)
@@
 	(wire
 		(pts
+			(xy 149.86 60.96) (xy 149.86 63.5)
+		)
+		(stroke
+			(width 0)
+			(type default)
+		)
+	)
+	(wire
+		(pts
 			(xy 157.48 109.22) (xy 157.48 114.3)
 		)
@@
 	(wire
 		(pts
-			(xy 154.94 53.34) (xy 152.4 53.34)
-		)
-		(stroke
-			(width 0)
-			(type default)
-		)
-	)
-	(wire
-		(pts
 			(xy 115.57 54.61) (xy 111.76 54.61)
 		)
@@
 	(wire
 		(pts
+			(xy 154.94 60.96) (xy 152.4 60.96)
+		)
+		(stroke
+			(width 0)
+			(type default)
+		)
+	)
+	(wire
+		(pts
 			(xy 130.81 93.98) (xy 139.7 93.98)
 		)
@@
 	(wire
 		(pts
-			(xy 149.86 53.34) (xy 149.86 63.5)
+			(xy 154.94 63.5) (xy 154.94 60.96)
 		)
 		(stroke
@@
 	(wire
 		(pts
-			(xy 154.94 63.5) (xy 154.94 53.34)
-		)
-		(stroke
-			(width 0)
-			(type default)
-		)
-	)
-	(wire
-		(pts
 			(xy 170.18 92.71) (xy 168.91 92.71)
 		)
@@
 		(pts
 			(xy 165.1 78.74) (xy 168.91 78.74)
+		)
+		(stroke
+			(width 0)
+			(type default)
+		)
+	)
+	(wire
+		(pts
+			(xy 152.4 60.96) (xy 149.86 60.96)
 		)
 		(stroke
@@
 			)
 			(justify left bottom)
+		)
+	)
+	(label "GND_Power"
+		(at 149.86 54.61 180)
+		(fields_autoplaced yes)
+		(effects
+			(font
+				(size 1.27 1.27)
+			)
+			(justify right bottom)
 		)
 	)
@@
 	)
 	(symbol
+		(lib_id "Motor:Motor_DC")
+		(at 209.55 59.69 0)
+		(unit 1)
+		(exclude_from_sim no)
+		(in_bom yes)
+		(on_board yes)
+		(dnp no)
+		(fields_autoplaced yes)
+		(property "Reference" "M1"
+			(at 214.63 60.9599 0)
+			(effects
+				(font
+					(size 1.27 1.27)
+				)
+				(justify left)
+			)
+		)
+		(property "Value" "Motor_DC"
+			(at 214.63 63.4999 0)
+			(effects
+				(font
+					(size 1.27 1.27)
+				)
+				(justify left)
+			)
+		)
+		(property "Footprint" "Connector_PinHeader_2.54mm:PinHeader_1x01_P2.54mm_Vertical"
+			(at 209.55 61.976 0)
+			(effects
+				(font
+					(size 1.27 1.27)
+				)
+				(hide yes)
+			)
+		)
+		(property "Datasheet" "~"
+			(at 209.55 61.976 0)
+			(effects
+				(font
+					(size 1.27 1.27)
+				)
+				(hide yes)
+			)
+		)
+		(property "Description" "DC Motor"
+			(at 209.55 59.69 0)
+			(effects
+				(font
+					(size 1.27 1.27)
+				)
+				(hide yes)
+			)
+		)
+		(pin "2"
+		)
+		(pin "1"
+		)
+		(instances
+			(project "CREPP.io"
+				(path "/8bcd0d00-b75f-4070-8d50-196a2022a31c/e5deda31-4de6-4c52-981c-0289ecc7c1e7"
+					(reference "M1")
+					(unit 1)
+				)
+			)
+		)
+	)
+	(symbol
+		(lib_id "CREPP_Drivers_Motors:L293D_THT")
+		(at 152.4 88.9 0)
+		(unit 1)
+		(exclude_from_sim no)
+		(in_bom yes)
+		(on_board yes)
+		(dnp no)
+		(fields_autoplaced yes)
+		(property "Reference" "U2"
+			(at 157.1341 60.96 0)
+			(effects
+				(font
+					(size 1.27 1.27)
+				)
+				(justify left)
+			)
+		)
+		(property "Value" "L293D"
+			(at 157.1341 63.5 0)
+			(effects
+				(font
+					(size 1.27 1.27)
+				)
+				(justify left)
+			)
+		)
+		(property "Footprint" "Package_DIP:DIP-16_W7.62mm_Socket"
+			(at 158.75 107.95 0)
+			(effects
+				(font
+					(size 1.27 1.27)
+				)
+				(justify left)
+				(hide yes)
+			)
+		)
+		(property "Datasheet" "http://www.ti.com/lit/ds/symlink/l293.pdf"
+			(at 144.78 71.12 0)
+			(effects
+				(font
+					(size 1.27 1.27)
+				)
+				(hide yes)
+			)
+		)
+		(property "Description" "Quadruple Half-H Drivers"
+			(at 152.4 88.9 0)
+			(effects
+				(font
+					(size 1.27 1.27)
+				)
+				(hide yes)
+			)
+		)
+		(pin "4"
+		)
+		(pin "16"
+		)
+		(pin "8"
+		)
+		(pin "6"
+		)
+		(pin "3"
+		)
+		(pin "9"
+		)
+		(pin "2"
+		)
+		(pin "1"
+		)
+		(pin "5"
+		)
+		(pin "7"
+		)
+		(pin "11"
+		)
+		(pin "14"
+		)
+		(pin "10"
+		)
+		(pin "13"
+		)
+		(pin "12"
+		)
+		(pin "15"
+		)
+		(instances
+			(project "CREPP.io"
+				(path "/8bcd0d00-b75f-4070-8d50-196a2022a31c/e5deda31-4de6-4c52-981c-0289ecc7c1e7"
+					(reference "U2")
+					(unit 1)
+				)
+			)
+		)
+	)
+	(symbol
 		(lib_id "Connector:Screw_Terminal_01x02")
 		(at 175.26 90.17 0)
@@
 				(path "/8bcd0d00-b75f-4070-8d50-196a2022a31c/e5deda31-4de6-4c52-981c-0289ecc7c1e7"
 					(reference "J11")
+					(unit 1)
+				)
+			)
+		)
+	)
+	(symbol
+		(lib_id "Motor:Motor_DC")
+		(at 210.82 78.74 0)
+		(unit 1)
+		(exclude_from_sim no)
+		(in_bom yes)
+		(on_board yes)
+		(dnp no)
+		(fields_autoplaced yes)
+		(property "Reference" "M2"
+			(at 215.9 80.0099 0)
+			(effects
+				(font
+					(size 1.27 1.27)
+				)
+				(justify left)
+			)
+		)
+		(property "Value" "Motor_DC"
+			(at 215.9 82.5499 0)
+			(effects
+				(font
+					(size 1.27 1.27)
+				)
+				(justify left)
+			)
+		)
+		(property "Footprint" "Connector_PinHeader_2.54mm:PinHeader_1x01_P2.54mm_Vertical"
+			(at 210.82 81.026 0)
+			(effects
+				(font
+					(size 1.27 1.27)
+				)
+				(hide yes)
+			)
+		)
+		(property "Datasheet" "~"
+			(at 210.82 81.026 0)
+			(effects
+				(font
+					(size 1.27 1.27)
+				)
+				(hide yes)
+			)
+		)
+		(property "Description" "DC Motor"
+			(at 210.82 78.74 0)
+			(effects
+				(font
+					(size 1.27 1.27)
+				)
+				(hide yes)
+			)
+		)
+		(pin "2"
+		)
+		(pin "1"
+		)
+		(instances
+			(project "CREPP.io"
+				(path "/8bcd0d00-b75f-4070-8d50-196a2022a31c/e5deda31-4de6-4c52-981c-0289ecc7c1e7"
+					(reference "M2")
 					(unit 1)
 				)
@@
 					(unit 1)
 				)
-			)
-		)
-	)
-	(symbol
-		(lib_id "Driver_Motor:L293D")
-		(at 152.4 88.9 0)
-		(unit 1)
-		(exclude_from_sim no)
-		(in_bom yes)
-		(on_board yes)
-		(dnp no)
-		(fields_autoplaced yes)
-		(property "Reference" "U2"
-			(at 157.1341 60.96 0)
-			(effects
-				(font
-					(size 1.27 1.27)
-				)
-				(justify left)
-			)
-		)
-		(property "Value" "L293D"
-			(at 157.1341 63.5 0)
-			(effects
-				(font
-					(size 1.27 1.27)
-				)
-				(justify left)
-			)
-		)
-		(property "Footprint" "Package_DIP:DIP-16_W7.62mm_Socket"
-			(at 158.75 107.95 0)
-			(effects
-				(font
-					(size 1.27 1.27)
-				)
-				(justify left)
-				(hide yes)
-			)
-		)
-		(property "Datasheet" "http://www.ti.com/lit/ds/symlink/l293.pdf"
-			(at 144.78 71.12 0)
-			(effects
-				(font
-					(size 1.27 1.27)
-				)
-				(hide yes)
-			)
-		)
-		(property "Description" "Quadruple Half-H Drivers"
-			(at 152.4 88.9 0)
-			(effects
-				(font
-					(size 1.27 1.27)
-				)
-				(hide yes)
-			)
-		)
-		(pin "13"
-		)
-		(pin "8"
-		)
-		(pin "7"
-		)
-		(pin "1"
-		)
-		(pin "12"
-		)
-		(pin "11"
-		)
-		(pin "10"
-		)
-		(pin "3"
-		)
-		(pin "4"
-		)
-		(pin "6"
-		)
-		(pin "5"
-		)
-		(pin "9"
-		)
-		(pin "14"
-		)
-		(pin "2"
-		)
-		(pin "16"
-		)
-		(pin "15"
-		)
-		(instances
-			(project "CREPP.io"
-				(path "/8bcd0d00-b75f-4070-8d50-196a2022a31c/e5deda31-4de6-4c52-981c-0289ecc7c1e7"
-					(reference "U2")
-					(unit 1)
-				)
