File: PCB/V2.0/Modules/I2C_Interface.kicad_sch (KiCad schematic)
At the start: 3 parts, among them J10 Power_Selector, J8 ST_PH_B4B-PH-K_1x04_P2.00mm, J9 ST_PH_B4B-PH-K_1x04_P2.00mm

Commit message: Add img
Parts:
- removed J8, J9: ST_PH_B4B-PH-K_1x04_P2.00mm, Connector_JST:JST_PH_B4B-PH-K_1x04_P2.00mm_Vertical, symbol Connector:Conn_01x04_Socket
- added J35, J8: Coon_01x04_Pin_2mm, Connector_JST:JST_PH_B4B-PH-K_1x04_P2.00mm_Vertical, symbol CREPP_Connectors_2mm:Conn_01x04_Pin_JST
Connections:
- net GND: now also J35.4 (Pin_4), J8.4 (Pin_4)
- net SCL: now also J35.2 (Pin_2), J8.2 (Pin_2)
- net SDA: now also J35.3 (Pin_3), J8.3 (Pin_3)
- net VCC_Common: now also J35.1 (Pin_1), J8.1 (Pin_1)
Changed lines of the file:
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@@
 	)
 	(symbol
-		(lib_id "Connector:Conn_01x04_Socket")
-		(at 168.91 63.5 0)
+		(lib_id "CREPP_Connectors_2mm:Conn_01x04_Pin_JST")
+		(at 168.91 80.01 0)
+		(mirror y)
 		(unit 1)
 		(exclude_from_sim no)
@@
 		(on_board yes)
 		(dnp no)
-		(property "Reference" "J9"
-			(at 170.434 62.992 0)
-			(effects
-				(font
-					(size 1.27 1.27)
-				)
-				(justify left)
-			)
-		)
-		(property "Value" "ST_PH_B4B-PH-K_1x04_P2.00mm"
-			(at 170.434 65.532 0)
-			(effects
-				(font
-					(size 1.27 1.27)
-				)
-				(justify left)
+		(property "Reference" "J8"
+			(at 170.18 82.5501 0)
+			(effects
+				(font
+					(size 1.27 1.27)
+				)
+				(justify right)
+			)
+		)
+		(property "Value" "Coon_01x04_Pin_2mm"
+			(at 170.18 80.0101 0)
+			(effects
+				(font
+					(size 1.27 1.27)
+				)
+				(justify right)
 			)
 		)
 		(property "Footprint" "Connector_JST:JST_PH_B4B-PH-K_1x04_P2.00mm_Vertical"
-			(at 168.91 63.5 0)
+			(at 168.91 80.01 0)
 			(effects
 				(font
@@
 		)
 		(property "Datasheet" "~"
-			(at 168.91 63.5 0)
+			(at 168.91 80.01 0)
 			(effects
 				(font
@@
 		)
 		(property "Description" "Generic connector, single row, 01x04, script generated"
-			(at 168.91 63.5 0)
-			(effects
-				(font
-					(size 1.27 1.27)
-				)
-				(hide yes)
-			)
+			(at 168.91 80.01 0)
+			(effects
+				(font
+					(size 1.27 1.27)
+				)
+				(hide yes)
+			)
+		)
+		(pin "4"
+		)
+		(pin "3"
+		)
+		(pin "2"
 		)
 		(pin "1"
-		)
-		(pin "4"
-		)
-		(pin "3"
-		)
-		(pin "2"
 		)
 		(instances
 			(project "CREPP.io"
 				(path "/8bcd0d00-b75f-4070-8d50-196a2022a31c/c4fb65bd-53fe-465d-8813-dbd5961ee741"
-					(reference "J9")
+					(reference "J8")
 					(unit 1)
 				)
@@
 	)
 	(symbol
-		(lib_id "Connector:Conn_01x04_Socket")
-		(at 168.91 80.01 0)
+		(lib_id "CREPP_Connectors_2mm:Conn_01x04_Pin_JST")
+		(at 168.91 63.5 0)
+		(mirror y)
 		(unit 1)
 		(exclude_from_sim no)
@@
 		(on_board yes)
 		(dnp no)
-		(property "Reference" "J8"
-			(at 170.942 76.454 0)
-			(effects
-				(font
-					(size 1.27 1.27)
-				)
-				(justify left)
-			)
-		)
-		(property "Value" "ST_PH_B4B-PH-K_1x04_P2.00mm"
-			(at 171.196 80.01 0)
-			(effects
-				(font
-					(size 1.27 1.27)
-				)
-				(justify left)
+		(property "Reference" "J35"
+			(at 170.18 66.0401 0)
+			(effects
+				(font
+					(size 1.27 1.27)
+				)
+				(justify right)
+			)
+		)
+		(property "Value" "Coon_01x04_Pin_2mm"
+			(at 170.18 63.5001 0)
+			(effects
+				(font
+					(size 1.27 1.27)
+				)
+				(justify right)
 			)
 		)
 		(property "Footprint" "Connector_JST:JST_PH_B4B-PH-K_1x04_P2.00mm_Vertical"
-			(at 168.91 80.01 0)
+			(at 168.91 63.5 0)
 			(effects
 				(font
@@
 		)
 		(property "Datasheet" "~"
-			(at 168.91 80.01 0)
+			(at 168.91 63.5 0)
 			(effects
 				(font
@@
 		)
 		(property "Description" "Generic connector, single row, 01x04, script generated"
-			(at 168.91 80.01 0)
-			(effects
-				(font
-					(size 1.27 1.27)
-				)
-				(hide yes)
-			)
+			(at 168.91 63.5 0)
+			(effects
+				(font
+					(size 1.27 1.27)
+				)
+				(hide yes)
+			)
+		)
+		(pin "4"
+		)
+		(pin "3"
+		)
+		(pin "2"
 		)
 		(pin "1"
-		)
-		(pin "4"
-		)
-		(pin "3"
-		)
-		(pin "2"
 		)
 		(instances
 			(project "CREPP.io"
 				(path "/8bcd0d00-b75f-4070-8d50-196a2022a31c/c4fb65bd-53fe-465d-8813-dbd5961ee741"
-					(reference "J8")
+					(reference "J35")
 					(unit 1)
 				)

Commit message: Update board
Parts:
- removed J10: Power_Selector, Connector_PinHeader_2.54mm:PinHeader_1x03_P2.54mm_Vertical, symbol Connector:Conn_01x03_Pin
- removed J35: Coon_01x04_Pin_2mm, Connector_JST:JST_PH_B4B-PH-K_1x04_P2.00mm_Vertical, symbol CREPP_Connectors_2mm:Conn_01x04_Pin_JST
- added J9: Coon_01x04_Pin_2mm, Connector_JST:JST_PH_B4B-PH-K_1x04_P2.00mm_Vertical, symbol CREPP_Connectors_2mm:Conn_01x04_Pin_JST
Connections:
- net VCC_Common is gone; now on net GND: J8.1 (Pin_1)
- net +3.3V: now also J8.4 (Pin_4), J9.4 (Pin_4)
- net GND: now also J9.1 (Pin_1); no longer J8.4 (Pin_4)
- net SCL: now also J8.3 (Pin_3), J9.3 (Pin_3); no longer J8.2 (Pin_2)
- net SDA: now also J8.2 (Pin_2), J9.2 (Pin_2); no longer J8.3 (Pin_3)

Commit message: Update
Parts:
- renumbered J9 to J2
Changed lines of the file:
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@@
 		(dnp no)
 		(fields_autoplaced yes)
-		(property "Reference" "J9"
+		(property "Reference" "J2"
 			(at 170.18 63.4999 0)
 			(effects
@@
 		)
 		(instances
-			(project ""
+			(project "CREPP.io"
 				(path "/8bcd0d00-b75f-4070-8d50-196a2022a31c/c4fb65bd-53fe-465d-8813-dbd5961ee741"
-					(reference "J9")
+					(reference "J2")
 					(unit 1)
 				)
