File: PCB/V2.0/Modules/IO_Extender.kicad_sch (KiCad schematic)
At the start: 9 parts, among them J20 GND_Analog, J21 +3.3V_Analog, J26 Addr_Selector, T1 TestPoint, U1 ADS1115IDGS

Commit message: Add RTC
Parts:
- removed C1: 100nF, Capacitor_SMD:C_0603_1608Metric, symbol Device:C
- removed J20: GND_Analog, Connector_PinHeader_2.54mm:PinHeader_1x04_P2.54mm_Vertical, symbol Connector:Conn_01x04_Socket
- removed J21: +3.3V_Analog, Connector_PinHeader_2.54mm:PinHeader_1x04_P2.54mm_Vertical, symbol Connector:Conn_01x04_Socket
- removed J26: Addr_Selector, Connector_PinHeader_2.54mm:PinHeader_1x03_P2.54mm_Vertical, symbol Connector:Conn_01x03_Pin
- removed JP1: J2.54MM, Connector_PinHeader_2.54mm:PinHeader_2x01_P2.54mm_Vertical, symbol Jumper:Jumper_2_Bridged
- removed R10, R16: 10k, Resistor_THT:R_Axial_DIN0207_L6.3mm_D2.5mm_P7.62mm_Horizontal, symbol Device:R
- removed T1: TestPoint, TestPoint:TestPoint_Pad_1.0x1.0mm, symbol Connector:TestPoint
- removed U1: ADS1115IDGS, Package_SO:TSSOP-10_3x3mm_P0.5mm, symbol Analog_ADC:ADS1115IDGS
Connections:
- no-connect marks 2 -> 0

Commit message: Update
Parts:
- added U12: PCA9635, Package_SO:TSSOP-28_4.4x9.7mm_P0.65mm, symbol Driver_LED:PCA9635
Connections:
- new net +3.3V: U12.28 (VDD)
- new net GND: U12.14 (VSS)
- new net LED_1: U12.9 (LED3)
- new net LED_2: U12.10 (LED4)
- new net LED_3: U12.11 (LED5)
- new net LED_4: U12.12 (LED6)
- new net LED_5: U12.13 (LED7)
- new net SCL: U12.26 (SCL)
- new net SDA: U12.27 (SDA)
- new net SERVO_1: U12.6 (LED0)
- new net SERVO_2: U12.7 (LED1)
- new net SERVO_3: U12.8 (LED2)
