File: PCB/V2.0/Modules/LED.kicad_sch (KiCad schematic)
At the start: 6 parts

Commit message: Add RTC
Parts:
- R6, R7, R8: footprint Resistor_THT:R_Axial_DIN0207_L6.3mm_D2.5mm_P7.62mm_Horizontal -> Resistor_THT:R_Axial_DIN0207_L6.3mm_D2.5mm_P10.16mm_Horizontal
Changed lines of the file:
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@@
 			)
 		)
-		(property "Footprint" "Resistor_THT:R_Axial_DIN0207_L6.3mm_D2.5mm_P7.62mm_Horizontal"
+		(property "Footprint" "Resistor_THT:R_Axial_DIN0207_L6.3mm_D2.5mm_P10.16mm_Horizontal"
 			(at 121.412 77.47 90)
 			(effects
@@
 			)
 		)
-		(property "Footprint" "Resistor_THT:R_Axial_DIN0207_L6.3mm_D2.5mm_P7.62mm_Horizontal"
+		(property "Footprint" "Resistor_THT:R_Axial_DIN0207_L6.3mm_D2.5mm_P10.16mm_Horizontal"
 			(at 134.112 77.47 90)
 			(effects
@@
 			)
 		)
-		(property "Footprint" "Resistor_THT:R_Axial_DIN0207_L6.3mm_D2.5mm_P7.62mm_Horizontal"
+		(property "Footprint" "Resistor_THT:R_Axial_DIN0207_L6.3mm_D2.5mm_P10.16mm_Horizontal"
 			(at 107.442 77.47 90)
 			(effects

Commit message: Update
Parts:
- removed D1, D2, D3: LED, LED_THT:LED_D5.0mm, symbol Device:LED
- added D1, D9: LED_Red, CREPP_LEDs:LED_D5.0mm_Red, symbol CREPP_LED:LED_5mm_THT
- added D10, D3, D4: LED_Green, CREPP_LEDs:LED_D5.0mm_Green, symbol CREPP_LED:LED_5mm_THT
- added D11, D2: LED_Orange, CREPP_LEDs:LED_D5.0mm_Orange, symbol CREPP_LED:LED_5mm_THT
- added R12, R13, R14, R5: 270, Resistor_THT:R_Axial_DIN0207_L6.3mm_D2.5mm_P10.16mm_Horizontal, symbol Device:R
Connections:
- net GND: now also D1.1 (K), D10.1 (K), D11.1 (K), D2.1 (K), D3.1 (K), D4.1 (K), D9.1 (K)
- net at R7.2: now also D1.2 (A)
- net at R8.2: now also D3.2 (A)
- net at R6.2: now also D11.2 (A)
- net GREEN renamed DEFAULT_LED
- net ORANGE_LED renamed L4
- net RED_LED renamed L3
- new net: D2.2 (A), R14.2
- new net: D9.2 (A), R12.2
- new net: D10.2 (A), R13.2
- new net: D4.2 (A), R5.2
- new net +5V: R5.1
- new net L1: R13.1
- new net L2: R14.1
- new net L5: R12.1
Other:
- moved on the sheet: R6, R8
