File: PCB/V2.0/Modules/Sensors.kicad_sch (KiCad schematic)
At the start: 8 parts, among them J2 HC-SR04_VIRTUAL, J23 HC-SR, J24 BME_VIRTUAL, J25 BME, J27 SIG_HCSR04, J36 Power_Selector

Commit message: Add RTC
Parts:
- R15: footprint Resistor_THT:R_Axial_DIN0207_L6.3mm_D2.5mm_P7.62mm_Horizontal -> Resistor_THT:R_Axial_DIN0207_L6.3mm_D2.5mm_P10.16mm_Horizontal
Changed lines of the file:
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@@
 			)
 		)
-		(property "Footprint" "Resistor_THT:R_Axial_DIN0207_L6.3mm_D2.5mm_P7.62mm_Horizontal"
+		(property "Footprint" "Resistor_THT:R_Axial_DIN0207_L6.3mm_D2.5mm_P10.16mm_Horizontal"
 			(at 24.892 59.69 90)
 			(effects

Commit message: update
Parts:
- removed J24: BME_VIRTUAL, Connector_PinSocket_2.54mm:PinSocket_1x06_P2.54mm_Vertical, symbol Connector:Conn_01x06_Socket
- added U10: ~, CREPP_Temperature_sensors:BME280_Breakout, symbol CREPP_Temperature_sensors:BME280_Breakout
Connections:
- no-connect marks 12 -> 6
Changed lines of the file:
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@@
-	)
-	(no_connect
-		(at 133.35 80.01)
-	)
-	(no_connect
-		(at 133.35 77.47)
 	)
 	(no_connect
@@
 	)
 	(no_connect
-		(at 133.35 67.31)
-	)
-	(no_connect
-		(at 133.35 72.39)
-	)
-	(no_connect
 		(at 119.38 66.04)
-	)
-	(no_connect
-		(at 133.35 69.85)
-	)
-	(no_connect
-		(at 133.35 74.93)
 	)
 	(no_connect
@@
 	)
 	(symbol
-		(lib_id "Connector:Conn_01x06_Socket")
-		(at 138.43 72.39 0)
+		(lib_id "CREPP_Temperature_sensors:BME280_Breakout")
+		(at 140.97 69.85 0)
 		(unit 1)
 		(exclude_from_sim no)
@@
 		(dnp no)
 		(fields_autoplaced yes)
-		(property "Reference" "J24"
-			(at 139.7 72.3899 0)
+		(property "Reference" "U10"
+			(at 152.4 71.1199 0)
 			(effects
 				(font
@@
 			)
 		)
-		(property "Value" "BME_VIRTUAL"
-			(at 139.7 74.9299 0)
+		(property "Value" "~"
+			(at 152.4 73.025 0)
 			(effects
 				(font
@@
 			)
 		)
-		(property "Footprint" "Connector_PinSocket_2.54mm:PinSocket_1x06_P2.54mm_Vertical"
-			(at 138.43 72.39 0)
+		(property "Footprint" "CREPP_Temperature_sensors:BME280_Breakout"
+			(at 140.97 69.85 0)
 			(effects
 				(font
@@
 			)
 		)
-		(property "Datasheet" "~"
-			(at 138.43 72.39 0)
+		(property "Datasheet" ""
+			(at 140.97 69.85 0)
 			(effects
 				(font
@@
 			)
 		)
-		(property "Description" "Generic connector, single row, 01x06, script generated"
-			(at 138.43 72.39 0)
+		(property "Description" ""
+			(at 140.97 69.85 0)
 			(effects
 				(font
@@
 				(hide yes)
 			)
-		)
-		(pin "4"
-		)
-		(pin "3"
-		)
-		(pin "2"
-		)
-		(pin "1"
-		)
-		(pin "6"
-		)
-		(pin "5"
 		)
 		(instances
 			(project "CREPP.io"
 				(path "/8bcd0d00-b75f-4070-8d50-196a2022a31c/54d9552b-b3ac-4100-8efe-05319c4e6125"
-					(reference "J24")
+					(reference "U10")
 					(unit 1)
 				)

Commit message: Update board
Changed lines of the file:
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@@
+		)
+	)
+	(label "GND"
+		(at 116.84 76.2 180)
+		(effects
+			(font
+				(size 1.27 1.27)
+			)
+			(justify right bottom)
 		)
 	)
 	(label "VCC_Sensor"
 		(at 128.27 100.33 0)
-		(fields_autoplaced yes)
 		(effects
 			(font
@@
 	(label "+5V"
 		(at 25.4 31.75 180)
-		(fields_autoplaced yes)
 		(effects
 			(font
@@
 	(label "+3.3V"
 		(at 132.08 95.25 0)
-		(fields_autoplaced yes)
 		(effects
 			(font
@@
 		)
 	)
-	(label "+3.3V"
-		(at 92.71 34.29 180)
-		(fields_autoplaced yes)
+	(label "VCC_Sensor"
+		(at 116.84 78.74 180)
 		(effects
 			(font
@@
 		)
 	)
-	(label "GND"
-		(at 116.84 76.2 180)
-		(fields_autoplaced yes)
+	(label "+3.3V"
+		(at 92.71 34.29 180)
 		(effects
 			(font
@@
 	(label "GND"
 		(at 26.67 25.4 180)
-		(fields_autoplaced yes)
+		(effects
+			(font
+				(size 1.27 1.27)
+			)
+			(justify right bottom)
+		)
+	)
+	(label "SDA"
+		(at 107.95 71.12 0)
+		(effects
+			(font
+				(size 1.27 1.27)
+			)
+			(justify left bottom)
+		)
+	)
+	(label "+5V"
+		(at 124.46 95.25 180)
+		(effects
+			(font
+				(size 1.27 1.27)
+			)
+			(justify right bottom)
+		)
+	)
+	(label "+3.3V"
+		(at 26.67 29.21 180)
+		(effects
+			(font
+				(size 1.27 1.27)
+			)
+			(justify right bottom)
+		)
+	)
+	(label "GND"
+		(at 92.71 26.67 180)
+		(effects
+			(font
+				(size 1.27 1.27)
+			)
+			(justify right bottom)
+		)
+	)
+	(label "+3.3V"
+		(at 26.67 54.61 180)
+		(effects
+			(font
+				(size 1.27 1.27)
+			)
+			(justify right bottom)
+		)
+	)
+	(label "GND"
+		(at 26.67 77.47 180)
 		(effects
 			(font
@@
 	(label "SCL"
 		(at 107.95 73.66 0)
-		(fields_autoplaced yes)
 		(effects
 			(font
@@
 		)
 	)
-	(label "SDA"
-		(at 107.95 71.12 0)
-		(fields_autoplaced yes)
+	(hierarchical_label "{I2C0}"
+		(shape input)
+		(at 95.25 59.69 180)
 		(effects
 			(font
 				(size 1.27 1.27)
 			)
-			(justify left bottom)
-		)
-	)
-	(label "+5V"
-		(at 124.46 95.25 180)
-		(fields_autoplaced yes)
-		(effects
-			(font
-				(size 1.27 1.27)
-			)
-			(justify right bottom)
-		)
-	)
-	(label "+3.3V"
-		(at 26.67 29.21 180)
-		(fields_autoplaced yes)
-		(effects
-			(font
-				(size 1.27 1.27)
-			)
-			(justify right bottom)
-		)
-	)
-	(label "GND"
-		(at 92.71 26.67 180)
-		(fields_autoplaced yes)
-		(effects
-			(font
-				(size 1.27 1.27)
-			)
-			(justify right bottom)
-		)
-	)
-	(label "+3.3V"
-		(at 26.67 54.61 180)
-		(fields_autoplaced yes)
-		(effects
-			(font
-				(size 1.27 1.27)
-			)
-			(justify right bottom)
-		)
-	)
-	(label "GND"
-		(at 26.67 77.47 180)
-		(fields_autoplaced yes)
-		(effects
-			(font
-				(size 1.27 1.27)
-			)
-			(justify right bottom)
-		)
-	)
-	(label "VCC_Sensor"
-		(at 116.84 78.74 180)
-		(fields_autoplaced yes)
-		(effects
-			(font
-				(size 1.27 1.27)
-			)
-			(justify right bottom)
+			(justify right)
 		)
 	)
@@
 		(shape output)
 		(at 39.37 64.77 0)
-		(fields_autoplaced yes)
 		(effects
 			(font
@@
 		)
 	)
-	(hierarchical_label "{I2C}"
+	(hierarchical_label "+5V"
 		(shape input)
-		(at 95.25 59.69 180)
-		(fields_autoplaced yes)
+		(at 30.48 31.75 0)
 		(effects
 			(font
 				(size 1.27 1.27)
 			)
-			(justify right)
+			(justify left)
 		)
 	)
-	(hierarchical_label "+5V"
+	(hierarchical_label "+3.3V"
 		(shape input)
-		(at 30.48 31.75 0)
-		(fields_autoplaced yes)
+		(at 30.48 29.21 0)
 		(effects
 			(font
@@
 		(shape passive)
 		(at 30.48 25.4 0)
-		(fields_autoplaced yes)
 		(effects
 			(font
-				(size 1.27 1.27)
-			)
-			(justify left)
-		)
-	)
-	(hierarchical_label "+3.3V"
-		(shape input)
-		(at 30.48 29.21 0)
-		(fields_autoplaced yes)
-		(effects
-			(font

Commit message: Update
Parts:
- removed J2: HC-SR04_VIRTUAL, Connector_PinSocket_2.54mm:PinSocket_1x04_P2.54mm_Vertical, symbol Connector:Conn_01x04_Socket
- removed J23: HC-SR, Connector_PinSocket_2.54mm:PinSocket_1x04_P2.54mm_Vertical, symbol Connector:Conn_01x04_Socket
- removed J27: SIG_HCSR04, Connector_PinHeader_2.54mm:PinHeader_1x02_P2.54mm_Vertical, symbol Connector:Conn_01x02_Pin
Connections:
- no-connect marks 6 -> 2
